File: PCB/VORTAC/KiCAD/VORTAC/Logic.sch (KiCad schematic (older format))
At the start: 76 parts, among them Q1 Q_PMOS_GSD, Q2 Q_NMOS_GSD, Q3 WSD4066DN, Q4 Q_NMOS_GSD, Q5 WSD4066DN, Q6 Q_PNP_BEC, Q7 Q_NPN_BEC, U1 TLV73333PDBV, U3 TPS54335ADRCR, U4 TPS54335ADRCR

Commit message: Holiday Break <3
Parts:
- added C49: 0.1uF 16V, Capacitor_SMD:C_0402_1005Metric, symbol Device:C_Small
- added R51, R52: 10K, Resistor_SMD:R_0402_1005Metric, symbol Device:R_Small
- C2: footprint Capacitor_SMD:C_0603_1608Metric -> Capacitor_SMD:C_0402_1005Metric; LCSC C66501 -> C1525
- gave numbers to parts that had none: 15
Connections:
- net +3V3: now also R52.1
- net GND: now also C49.1
- new net TOOL_ID: C49.2, R51.2, R52.2
- new net TOOL_ID_PIN: R51.1
Changed lines of the file:
@@
 F 0 "C2" H 10050 6100 50  0000 L CNN
 F 1 "0.1uF 16V" H 10050 6000 50  0000 L CNN
-F 2 "Capacitor_SMD:C_0603_1608Metric" H 9950 6100 50  0001 C CNN
-F 3 "https://www.lcsc.com/product-detail/Multilayer-Ceramic-Capacitors-MLCC-SMD-SMT_Samsung-Electro-Mechanics-CL10B104KO8NNNC_C66501.html" H 9950 6100 50  0001 C CNN
-F 4 "C66501" H 9950 6100 50  0001 C CNN "LCSC"
+F 2 "Capacitor_SMD:C_0402_1005Metric" H 9950 6100 50  0001 C CNN
+F 3 "https://www.lcsc.com/product-detail/Multilayer-Ceramic-Capacitors-MLCC-SMD-SMT_Samsung-Electro-Mechanics-CL05B104KO5NNNC_C1525.html" H 9950 6100 50  0001 C CNN
+F 4 "C1525" H 9950 6100 50  0001 C CNN "LCSC"
 	1    9950 6100
 	1    0    0    -1
@@
 FAN_1_TACHO_PIN
 $Comp
-L power:+3.3V #PWR?
+L power:+3.3V #PWR0148
 U 1 1 61BDF3BD
 P 7100 850
-F 0 "#PWR?" H 7100 700 50  0001 C CNN
+F 0 "#PWR0148" H 7100 700 50  0001 C CNN
 F 1 "+3.3V" V 7115 978 50  0000 L CNN
 F 2 "" H 7100 850 50  0001 C CNN
@@
 $EndComp
 $Comp
-L Device:R_Small R?
+L Device:R_Small R39
 U 1 1 61BE38C7
 P 6550 1050
-F 0 "R?" V 6650 1050 50  0000 C CNN
+F 0 "R39" V 6650 1050 50  0000 C CNN
 F 1 "10K" V 6450 1050 50  0000 C CNN
 F 2 "Resistor_SMD:R_0402_1005Metric" H 6550 1050 50  0001 C CNN
@@
 $EndComp
 $Comp
-L Device:R_Small R?
+L Device:R_Small R45
 U 1 1 61BEFC13
 P 6900 850
-F 0 "R?" V 7000 850 50  0000 C CNN
+F 0 "R45" V 7000 850 50  0000 C CNN
 F 1 "10K" V 6800 850 50  0000 C CNN
 F 2 "Resistor_SMD:R_0402_1005Metric" H 6900 850 50  0001 C CNN
@@
 FAN_2_TACHO_PIN
 $Comp
-L power:+3.3V #PWR?
+L power:+3.3V #PWR0164
 U 1 1 61CB33CC
 P 7100 1350
-F 0 "#PWR?" H 7100 1200 50  0001 C CNN
+F 0 "#PWR0164" H 7100 1200 50  0001 C CNN
 F 1 "+3.3V" V 7115 1478 50  0000 L CNN
 F 2 "" H 7100 1350 50  0001 C CNN
@@
 $EndComp
 $Comp
-L Device:R_Small R?
+L Device:R_Small R40
 U 1 1 61CB33D2
 P 6550 1550
-F 0 "R?" V 6650 1550 50  0000 C CNN
+F 0 "R40" V 6650 1550 50  0000 C CNN
 F 1 "10K" V 6450 1550 50  0000 C CNN
 F 2 "Resistor_SMD:R_0402_1005Metric" H 6550 1550 50  0001 C CNN
@@
 $EndComp
 $Comp
-L Device:R_Small R?
+L Device:R_Small R46
 U 1 1 61CB33D8
 P 6900 1350
-F 0 "R?" V 7000 1350 50  0000 C CNN
+F 0 "R46" V 7000 1350 50  0000 C CNN
 F 1 "10K" V 6800 1350 50  0000 C CNN
 F 2 "Resistor_SMD:R_0402_1005Metric" H 6900 1350 50  0001 C CNN
@@
 LED_1_PWM_PIN
 $Comp
-L power:+3.3V #PWR?
+L power:+3.3V #PWR0165
 U 1 1 61CC4D55
 P 7100 1850
-F 0 "#PWR?" H 7100 1700 50  0001 C CNN
+F 0 "#PWR0165" H 7100 1700 50  0001 C CNN
 F 1 "+3.3V" V 7115 1978 50  0000 L CNN
 F 2 "" H 7100 1850 50  0001 C CNN
@@
 $EndComp
 $Comp
-L Device:R_Small R?
+L Device:R_Small R41
 U 1 1 61CC4D5B
 P 6550 2050
-F 0 "R?" V 6650 2050 50  0000 C CNN
+F 0 "R41" V 6650 2050 50  0000 C CNN
 F 1 "10K" V 6450 2050 50  0000 C CNN
 F 2 "Resistor_SMD:R_0402_1005Metric" H 6550 2050 50  0001 C CNN
@@
 $EndComp
 $Comp
-L Device:R_Small R?
+L Device:R_Small R47
 U 1 1 61CC4D61
 P 6900 1850
-F 0 "R?" V 7000 1850 50  0000 C CNN
+F 0 "R47" V 7000 1850 50  0000 C CNN
 F 1 "10K" V 6800 1850 50  0000 C CNN
 F 2 "Resistor_SMD:R_0402_1005Metric" H 6900 1850 50  0001 C CNN
@@
 IO_1_OUT_PIN
 $Comp
-L Device:R_Small R?
+L Device:R_Small R42
 U 1 1 61CEB167
 P 6550 2700
-F 0 "R?" V 6650 2700 50  0000 C CNN
+F 0 "R42" V 6650 2700 50  0000 C CNN
 F 1 "10K" V 6450 2700 50  0000 C CNN
 F 2 "Resistor_SMD:R_0402_1005Metric" H 6550 2700 50  0001 C CNN
@@
 $EndComp
 $Comp
-L Device:R_Small R?
+L Device:R_Small R48
 U 1 1 61CEB16D
 P 6900 2500
-F 0 "R?" V 7000 2500 50  0000 C CNN
+F 0 "R48" V 7000 2500 50  0000 C CNN
 F 1 "10K" V 6800 2500 50  0000 C CNN
 F 2 "Resistor_SMD:R_0402_1005Metric" H 6900 2500 50  0001 C CNN
@@
 	7000 2500 7100 2500
 $Comp
-L power:+3.3V #PWR?
+L power:+3.3V #PWR0166
 U 1 1 61CEB161
 P 7100 2500
-F 0 "#PWR?" H 7100 2350 50  0001 C CNN
+F 0 "#PWR0166" H 7100 2350 50  0001 C CNN
 F 1 "+3.3V" V 7115 2628 50  0000 L CNN
 F 2 "" H 7100 2500 50  0001 C CNN
@@
 $EndComp
 $Comp
-L Device:C_Small C?
+L Device:C_Small C46
 U 1 1 61D71811
 P 6900 2900
-AR Path="/613DBE83/61D71811" Ref="C?"  Part="1"
+AR Path="/613DBE83/61D71811" Ref="C46"  Part="1"
 AR Path="/613DC005/61D71811" Ref="C?"  Part="1"
-F 0 "C?" V 7000 3050 50  0000 R CNN
+F 0 "C46" V 7000 3050 50  0000 R CNN
 F 1 "0.1uF 16V" V 7000 2800 50  0000 R CNN
 F 2 "Capacitor_SMD:C_0402_1005Metric" H 6900 2900 50  0001 C CNN
@@
 	7000 2900 7100 2900
 $Comp
-L power:GND #PWR?
+L power:GND #PWR0167
 U 1 1 61DC6F2F
 P 7100 2900
-F 0 "#PWR?" H 7100 2650 50  0001 C CNN
+F 0 "#PWR0167" H 7100 2650 50  0001 C CNN
 F 1 "GND" V 7105 2772 50  0000 R CNN
 F 2 "" H 7100 2900 50  0001 C CNN
@@
 IO_2_OUT_PIN
 $Comp
-L Device:R_Small R?
+L Device:R_Small R43
 U 1 1 61E4ABCF
 P 6550 3450
-F 0 "R?" V 6650 3450 50  0000 C CNN
+F 0 "R43" V 6650 3450 50  0000 C CNN
 F 1 "10K" V 6450 3450 50  0000 C CNN
 F 2 "Resistor_SMD:R_0402_1005Metric" H 6550 3450 50  0001 C CNN
@@
 $EndComp
 $Comp
-L Device:R_Small R?
+L Device:R_Small R49
 U 1 1 61E4ABD5
 P 6900 3250
-F 0 "R?" V 7000 3250 50  0000 C CNN
+F 0 "R49" V 7000 3250 50  0000 C CNN
 F 1 "10K" V 6800 3250 50  0000 C CNN
 F 2 "Resistor_SMD:R_0402_1005Metric" H 6900 3250 50  0001 C CNN
@@
 	7000 3250 7100 3250
 $Comp
-L power:+3.3V #PWR?
+L power:+3.3V #PWR0168
 U 1 1 61E4ABE0
 P 7100 3250
-F 0 "#PWR?" H 7100 3100 50  0001 C CNN
+F 0 "#PWR0168" H 7100 3100 50  0001 C CNN
 F 1 "+3.3V" V 7115 3378 50  0000 L CNN
 F 2 "" H 7100 3250 50  0001 C CNN
@@
 $EndComp
 $Comp
-L Device:C_Small C?
+L Device:C_Small C47
 U 1 1 61E4ABE7
 P 6900 3650
-AR Path="/613DBE83/61E4ABE7" Ref="C?"  Part="1"
+AR Path="/613DBE83/61E4ABE7" Ref="C47"  Part="1"
 AR Path="/613DC005/61E4ABE7" Ref="C?"  Part="1"
-F 0 "C?" V 7000 3800 50  0000 R CNN
+F 0 "C47" V 7000 3800 50  0000 R CNN
 F 1 "0.1uF 16V" V 7000 3550 50  0000 R CNN
 F 2 "Capacitor_SMD:C_0402_1005Metric" H 6900 3650 50  0001 C CNN
@@
 	7000 3650 7100 3650
 $Comp
-L power:GND #PWR?
+L power:GND #PWR0169
 U 1 1 61E4ABF0
 P 7100 3650
-F 0 "#PWR?" H 7100 3400 50  0001 C CNN
+F 0 "#PWR0169" H 7100 3400 50  0001 C CNN
 F 1 "GND" V 7105 3522 50  0000 R CNN
 F 2 "" H 7100 3650 50  0001 C CNN
@@
 IO_3_OUT_PIN
 $Comp
-L Device:R_Small R?
+L Device:R_Small R44
 U 1 1 61E5F586
 P 6550 4150
-F 0 "R?" V 6650 4150 50  0000 C CNN
+F 0 "R44" V 6650 4150 50  0000 C CNN
 F 1 "10K" V 6450 4150 50  0000 C CNN
 F 2 "Resistor_SMD:R_0402_1005Metric" H 6550 4150 50  0001 C CNN
@@
 $EndComp
 $Comp
-L Device:R_Small R?
+L Device:R_Small R50
 U 1 1 61E5F58C
 P 6900 3950
-F 0 "R?" V 7000 3950 50  0000 C CNN
+F 0 "R50" V 7000 3950 50  0000 C CNN
 F 1 "10K" V 6800 3950 50  0000 C CNN
 F 2 "Resistor_SMD:R_0402_1005Metric" H 6900 3950 50  0001 C CNN
@@
 	7000 3950 7100 3950
 $Comp
-L power:+3.3V #PWR?
+L power:+3.3V #PWR0170
 U 1 1 61E5F597
 P 7100 3950
-F 0 "#PWR?" H 7100 3800 50  0001 C CNN
+F 0 "#PWR0170" H 7100 3800 50  0001 C CNN
 F 1 "+3.3V" V 7115 4078 50  0000 L CNN
 F 2 "" H 7100 3950 50  0001 C CNN
@@
 $EndComp
 $Comp
-L Device:C_Small C?
+L Device:C_Small C48
 U 1 1 61E5F59E
 P 6900 4350
-AR Path="/613DBE83/61E5F59E" Ref="C?"  Part="1"
+AR Path="/613DBE83/61E5F59E" Ref="C48"  Part="1"
 AR Path="/613DC005/61E5F59E" Ref="C?"  Part="1"
-F 0 "C?" V 7000 4500 50  0000 R CNN
+F 0 "C48" V 7000 4500 50  0000 R CNN
 F 1 "0.1uF 16V" V 7000 4250 50  0000 R CNN
 F 2 "Capacitor_SMD:C_0402_1005Metric" H 6900 4350 50  0001 C CNN
@@
 	7000 4350 7100 4350
 $Comp
-L power:GND #PWR?
+L power:GND #PWR0171
 U 1 1 61E5F5A7
 P 7100 4350
-F 0 "#PWR?" H 7100 4100 50  0001 C CNN
+F 0 "#PWR0171" H 7100 4100 50  0001 C CNN
 F 1 "GND" V 7105 4222 50  0000 R CNN
 F 2 "" H 7100 4350 50  0001 C CNN
@@
 Wire Wire Line
 	6650 4150 7100 4150
+Text GLabel 6250 4900 0    50   Input ~ 0
+TOOL_ID
+Text GLabel 7100 4900 2    50   Input ~ 0
+TOOL_ID_PIN
+$Comp
+L Device:R_Small R51
+U 1 1 61F97E57
+P 6550 4900
+F 0 "R51" V 6650 4900 50  0000 C CNN
+F 1 "10K" V 6450 4900 50  0000 C CNN
+F 2 "Resistor_SMD:R_0402_1005Metric" H 6550 4900 50  0001 C CNN
+F 3 "~" H 6550 4900 50  0001 C CNN
+	1    6550 4900
+	0    1    1    0
+$EndComp
+$Comp
+L Device:R_Small R52
+U 1 1 61F97E5D
+P 6900 4700
+F 0 "R52" V 7000 4700 50  0000 C CNN
+F 1 "10K" V 6800 4700 50  0000 C CNN
+F 2 "Resistor_SMD:R_0402_1005Metric" H 6900 4700 50  0001 C CNN
+F 3 "~" H 6900 4700 50  0001 C CNN
+	1    6900 4700
+	0    1    1    0
+$EndComp
+Wire Wire Line
+	6350 4700 6350 4900
+Wire Wire Line
+	6350 4900 6450 4900
+Wire Wire Line
+	6350 4900 6250 4900
+Connection ~ 6350 4900
+Wire Wire Line
+	7000 4700 7100 4700
+$Comp
+L power:+3.3V #PWR0172
+U 1 1 61F97E68
+P 7100 4700
+F 0 "#PWR0172" H 7100 4550 50  0001 C CNN
+F 1 "+3.3V" V 7115 4828 50  0000 L CNN
+F 2 "" H 7100 4700 50  0001 C CNN
+F 3 "" H 7100 4700 50  0001 C CNN
+	1    7100 4700
+	0    1    1    0
+$EndComp
+$Comp
+L Device:C_Small C49
+U 1 1 61F97E6F
+P 6900 5100
+AR Path="/613DBE83/61F97E6F" Ref="C49"  Part="1"
+AR Path="/613DC005/61F97E6F" Ref="C?"  Part="1"
+F 0 "C49" V 7000 5250 50  0000 R CNN
+F 1 "0.1uF 16V" V 7000 5000 50  0000 R CNN
+F 2 "Capacitor_SMD:C_0402_1005Metric" H 6900 5100 50  0001 C CNN
+F 3 "https://www.lcsc.com/product-detail/Multilayer-Ceramic-Capacitors-MLCC-SMD-SMT_Samsung-Electro-Mechanics-CL05B104KO5NNNC_C1525.html" H 6900 5100 50  0001 C CNN
+F 4 "C1525" V 6900 5100 50  0001 C CNN "LCSC"
+	1    6900 5100
+	0    1    1    0
+$EndComp
+Wire Wire Line
+	6350 4900 6350 5100
+Wire Wire Line
+	6350 5100 6800 5100
+Wire Wire Line
+	7000 5100 7100 5100
+$Comp
+L power:GND #PWR0173
+U 1 1 61F97E78
+P 7100 5100
+F 0 "#PWR0173" H 7100 4850 50  0001 C CNN
+F 1 "GND" V 7105 4972 50  0000 R CNN
+F 2 "" H 7100 5100 50  0001 C CNN
+F 3 "" H 7100 5100 50  0001 C CNN
+	1    7100 5100
+	0    -1   -1   0
+$EndComp
+Wire Wire Line
+	6350 4700 6800 4700
+Wire Wire Line
+	6650 4900 7100 4900
 $EndSCHEMATC

Commit message: pushy
Parts:
- L1, L2: LCSC ALT (none) -> C436530
- U1: Field4 C134139 -> (none); LCSC (none) -> C408972
Changed lines of the file:
@@
 F 3 "https://www.lcsc.com/product-detail/Power-Inductors_Sunlord-MWSA0503S-100MT_C408412.html" H 3250 4600 50  0001 C CNN
 F 4 "C408412" V 3250 4600 50  0001 C CNN "LCSC"
+F 5 "C436530" V 3250 4600 50  0001 C CNN "LCSC ALT"
 	1    3250 4600
 	0    -1   -1   0
@@
 F 3 "https://www.lcsc.com/product-detail/Power-Inductors_Sunlord-MWSA0503S-100MT_C408412.html" H 3250 2600 50  0001 C CNN
 F 4 "C408412" V 3250 2600 50  0001 C CNN "LCSC"
+F 5 "C436530" V 3250 2600 50  0001 C CNN "LCSC ALT"
 	1    3250 2600
 	0    -1   -1   0
@@
 F 1 "TLV73333PDBV" H 1300 6550 50  0000 C CNN
 F 2 "Package_TO_SOT_SMD:SOT-23-5" H 1550 7325 50  0001 C CIN
-F 3 "https://www.lcsc.com/product-detail/Linear-Voltage-Regulators-LDO_Texas-Instruments-TLV73333PDBVR_C134139.html" H 1550 7000 50  0001 C CNN
-F 4 "C134139" H 1550 7000 50  0001 C CNN "Field4"
+F 3 "https://www.lcsc.com/product-detail/Linear-Voltage-Regulators-LDO_Texas-Instruments-TLV74333PDBVR_C408972.html" H 1550 7000 50  0001 C CNN
+F 4 "C408972" H 1550 7000 50  0001 C CNN "LCSC"
 	1    1550 7000
 	1    0    0    -1
