File: PCB/VORTAC/KiCAD/VORTAC/Headers.sch (KiCad schematic (older format))
At the start: 27 parts, among them J1 DEBUG, J10 FAN_01_V, J11 FAN_02_V, J12 LED_V, J13 THERM_R, J14 918-418K2023S40001, J15 STEPPER, J16 IO, J2 Molex Micro Fit 3.0, J3 MillMax_004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

Commit message: Routing WIP
Parts:
- removed JP1, JP2: SolderJumper_2_Bridged, ToolChanger:SolderJumper_Hex_Bridged_Pad, symbol Jumper:SolderJumper_2_Bridged
- removed JP3, JP4: SolderJumper_2_Open, ToolChanger:SolderJumper_Hex_Open_Pad, symbol Jumper:SolderJumper_2_Open
- added JP1: DATA_H JUMPER, Jumper:SolderJumper-3_P1.3mm_Bridged12_Pad1.0x1.5mm, symbol Jumper:SolderJumper_3_Bridged12
- added JP2: DATA_L JUMPER, Jumper:SolderJumper-3_P1.3mm_Bridged12_Pad1.0x1.5mm, symbol Jumper:SolderJumper_3_Bridged12
- J15: footprint Connector_JST:JST_PH_S4B-PH-K_1x04_P2.00mm_Horizontal -> ToolChanger:JST_PH_S4B-PH-K_1x04_P2.00mm_Horizontal
Connections:
- net labels added: +12V, +3.3V, +3.3VA, +5V, BOOT_1, DEBUG_SWCLK, DEBUG_SWDIO, DEBUG_SWO, DOCK_VDC, NRST, VDC
- net labels removed: 12V, 5V, AREF, DOCK_V_IN, V_IN
- wire segments 92 -> 104
Other:
- moved on the sheet: H1, H2, J1, J10, J11, J12

Commit message: Reversed voltage selectors to simplify routing
Parts:
- J1, J10, J11, J12: footprint Connector_PinHeader_1.27mm:PinHeader_2x03_P1.27mm_Vertical -> ToolChanger:PinHeader_2x03_P1.27mm_Vertical
- J13: footprint Connector_PinHeader_1.27mm:PinHeader_2x02_P1.27mm_Vertical -> ToolChanger:PinHeader_2x02_P1.27mm_Vertical
- J9: footprint Connector_JST:JST_PH_B2B-PH-K_1x02_P2.00mm_Vertical -> Connector_JST:JST_PH_B3B-PH-K_1x03_P2.00mm_Vertical; symbol Connector_Generic:Conn_01x02 -> Connector_Generic:Conn_01x03
Connections:
- net +12V: now also J10.3 (Pin_3), J11.3 (Pin_3), J12.3 (Pin_3); no longer J10.4 (Pin_4), J11.4 (Pin_4), J12.4 (Pin_4)
- net +5V: now also J10.5 (Pin_5), J11.5 (Pin_5), J12.5 (Pin_5); no longer J10.6 (Pin_6), J11.6 (Pin_6), J12.6 (Pin_6)
- net FAN_1_V_OUT: now also J10.2 (Pin_2), J10.4 (Pin_4), J10.6 (Pin_6); no longer J10.1 (Pin_1), J10.3 (Pin_3), J10.5 (Pin_5)
- net FAN_2_V_OUT: now also J11.2 (Pin_2), J11.4 (Pin_4), J11.6 (Pin_6); no longer J11.1 (Pin_1), J11.3 (Pin_3), J11.5 (Pin_5)
- net LED_1_V_OUT: now also J12.2 (Pin_2), J12.4 (Pin_4), J12.6 (Pin_6); no longer J12.1 (Pin_1), J12.3 (Pin_3), J12.5 (Pin_5)
- net VDC: now also J10.1 (Pin_1), J11.1 (Pin_1), J12.1 (Pin_1); no longer J10.2 (Pin_2), J11.2 (Pin_2), J12.2 (Pin_2)
- new net LED_1_PWM: J9.3 (Pin_3)
Other:
- moved on the sheet: J1, J10, J11, J12

Commit message: More Routing
Connections:
- net +3V3: now also J1.2 (Pin_2); no longer J1.5 (Pin_5)
- net BOOT_1: now also J1.1 (Pin_1); no longer J1.6 (Pin_6)
- net DEBUG_SWCLK: now also J1.6 (Pin_6); no longer J1.1 (Pin_1)
- net DEBUG_SWDIO: now also J1.5 (Pin_5); no longer J1.2 (Pin_2)
- net DOCK_GND: now also J2.1 (Pin_1); no longer J2.2 (Pin_2)
- net DOCK_VDC: now also J2.2 (Pin_2); no longer J2.3 (Pin_3)
- net GND: now also J1.4 (Pin_4), J2.3 (Pin_3), J3.2; no longer J1.3 (Pin_3), J2.1 (Pin_1), J3.5
- net IO_1_OUT: now also J16.5 (Pin_5); no longer J16.3 (Pin_3)
- net IO_3_OUT: now also J16.3 (Pin_3); no longer J16.5 (Pin_5)
- net NRST: now also J1.3 (Pin_3); no longer J1.4 (Pin_4)
- net TOOL_DATA_H: now also J3.4; no longer J4.4
- net TOOL_DATA_L: now also J3.5; no longer J4.5
- net TOOL_ID: now also J4.4; no longer J3.2
- net VDC: now also J3.3; no longer J3.4
Other:
- note added: "Maybe add boot pin for reflashing ability?"
- moved on the sheet: J12
Changed lines of the file:
@@
 $EndDescr
-$Comp
-L ToolChanger:MillMax_004 J4
-U 1 1 61450233
-P 2000 2675
-F 0 "J4" H 2180 2956 50  0000 L CNN
-F 1 "MillMax_004" H 2180 2865 50  0000 L CNN
-F 2 "ToolChanger:MillMax-858-10-004-10-012000" H 2270 2565 50  0001 C CNN
-F 3 "https://www.mouser.de/datasheet/2/273/MMMC_S_A0006083300_1-2558511.pdf" H 2270 2565 50  0001 C CNN
-F 4 "575-8582200480012101" H 2000 2675 50  0001 C CNN "Mouser"
-	1    2000 2675
-	1    0    0    -1
-$EndComp
 $Comp
 L power:GND #PWR02
@@
 $EndComp
 $Comp
-L power:GND #PWR03
-U 1 1 614656F6
-P 1750 1850
-F 0 "#PWR03" H 1750 1600 50  0001 C CNN
-F 1 "GND" V 1755 1722 50  0000 R CNN
-F 2 "" H 1750 1850 50  0001 C CNN
-F 3 "" H 1750 1850 50  0001 C CNN
-	1    1750 1850
-	0    1    1    0
-$EndComp
-$Comp
 L power:GND #PWR04
 U 1 1 61466537
@@
 	0    1    1    0
 $EndComp
-$Comp
-L power:GND #PWR05
-U 1 1 61466955
-P 1750 3100
-F 0 "#PWR05" H 1750 2850 50  0001 C CNN
-F 1 "GND" V 1755 2972 50  0000 R CNN
-F 2 "" H 1750 3100 50  0001 C CNN
-F 3 "" H 1750 3100 50  0001 C CNN
-	1    1750 3100
-	0    1    1    0
-$EndComp
-Text GLabel 1400 2900 0    50   Input ~ 0
+Text GLabel 1400 1650 0    50   Input ~ 0
 TOOL_DATA_L
-Text GLabel 1400 1200 0    50   Input ~ 0
+Text GLabel 1400 2750 0    50   Input ~ 0
 TOOL_ID
 $Comp
 L power:GND #PWR01
 U 1 1 61467CD1
-P 1400 1650
-F 0 "#PWR01" H 1400 1400 50  0001 C CNN
-F 1 "GND" V 1405 1522 50  0000 R CNN
-F 2 "" H 1400 1650 50  0001 C CNN
-F 3 "" H 1400 1650 50  0001 C CNN
-	1    1400 1650
-	0    1    1    0
-$EndComp
-Text GLabel 1400 3800 0    50   Input ~ 0
+P 1400 1200
+F 0 "#PWR01" H 1400 950 50  0001 C CNN
+F 1 "GND" V 1405 1072 50  0000 R CNN
+F 2 "" H 1400 1200 50  0001 C CNN
+F 3 "" H 1400 1200 50  0001 C CNN
+	1    1400 1200
+	0    1    1    0
+$EndComp
+Text GLabel 1400 3700 0    50   Input ~ 0
 DOCK_VDC
-$Comp
-L ToolChanger:MillMax_004 J3
-U 1 1 6144A490
-P 2000 1425
-F 0 "J3" H 2180 1706 50  0000 L CNN
-F 1 "MillMax_004" H 2180 1615 50  0000 L CNN
-F 2 "ToolChanger:MillMax-858-10-004-10-012000" H 2270 1315 50  0001 C CNN
-F 3 "https://www.mouser.de/datasheet/2/273/MMMC_S_A0006083300_1-2558511.pdf" H 2270 1315 50  0001 C CNN
-F 4 "575-8582200480012101" H 2000 1425 50  0001 C CNN "Mouser"
-	1    2000 1425
-	1    0    0    -1
-$EndComp
 Text Notes 2250 1500 0    50   ~ 0
 Upper Pogo Connector
@@
 Text Notes 850  850  0    71   ~ 0
 Tool Interface
-Text GLabel 1400 2750 0    50   Input ~ 0
+Text GLabel 1400 1500 0    50   Input ~ 0
 TOOL_DATA_H
 Text GLabel 2300 3600 2    50   Input ~ 0
@@
 Text Notes 9200 7050 0    50   ~ 0
 todo:\n- consider connector selection\n- consider combining fan or io/led headers\n- remove duplicate heater/thermistor header\n- add probepoints\n- change usb-c symbol (sucks bro)
-NoConn ~ 1400 1350
 Text GLabel 1600 4700 0    50   Input ~ 0
 HOST_USB_DRAIN
-Text GLabel 1400 3700 0    50   Input ~ 0
+Text GLabel 1400 3600 0    50   Input ~ 0
 DOCK_GND
 $Comp
@@
 	1400 1200 1750 1200
 Wire Wire Line
-	1750 1350 1400 1350
-Wire Wire Line
 	1400 1500 1750 1500
 Wire Wire Line
@@
 Wire Wire Line
 	2100 3600 2300 3600
-$Comp
-L power:GND #PWR0120
-U 1 1 61BCE37C
-P 1400 3600
-F 0 "#PWR0120" H 1400 3350 50  0001 C CNN
-F 1 "GND" V 1405 3472 50  0000 R CNN
-F 2 "" H 1400 3600 50  0001 C CNN
-F 3 "" H 1400 3600 50  0001 C CNN
-	1    1400 3600
-	0    1    1    0
-$EndComp
 Wire Wire Line
 	1400 2900 1750 2900
@@
 L power:VDC #PWR0136
 U 1 1 620C2CE2
-P 1400 1500
-F 0 "#PWR0136" H 1400 1400 50  0001 C CNN
-F 1 "VDC" V 1415 1627 50  0000 L CNN
-F 2 "" H 1400 1500 50  0001 C CNN
-F 3 "" H 1400 1500 50  0001 C CNN
-	1    1400 1500
+P 1400 1350
+F 0 "#PWR0136" H 1400 1250 50  0001 C CNN
+F 1 "VDC" V 1415 1477 50  0000 L CNN
+F 2 "" H 1400 1350 50  0001 C CNN
+F 3 "" H 1400 1350 50  0001 C CNN
+	1    1400 1350
 	0    -1   -1   0
 $EndComp
@@
 	1    0    0    -1
 $EndComp
-Text GLabel 7850 2350 0    50   Input ~ 0
+Text GLabel 7850 2550 0    50   Input ~ 0
 IO_1_OUT
 Text GLabel 7850 2450 0    50   Input ~ 0
 IO_2_OUT
-Text GLabel 7850 2550 0    50   Input ~ 0
+Text GLabel 7850 2350 0    50   Input ~ 0
 IO_3_OUT
 Wire Wire Line
@@
 Debug Header
 $Comp
-L Connector_Generic:Conn_02x03_Odd_Even J1
-U 1 1 618086B2
-P 8150 4100
-F 0 "J1" H 7900 4500 50  0000 C CNN
-F 1 "DEBUG" H 7900 4400 50  0000 C CNN
-F 2 "ToolChanger:PinHeader_2x03_P1.27mm_Vertical" H 8150 4100 50  0001 C CNN
-F 3 "~" H 8150 4100 50  0001 C CNN
-	1    8150 4100
-	1    0    0    -1
-$EndComp
-$Comp
 L Connector_Generic:Conn_02x02_Odd_Even J13
 U 1 1 61AA32CC
@@
 Wire Wire Line
 	6300 3500 6300 3400
-Text GLabel 6400 4500 2    50   Input ~ 0
+Text GLabel 6400 4450 2    50   Input ~ 0
 LED_1_V_OUT
 Wire Wire Line
-	5800 4600 5700 4600
-Wire Wire Line
-	5800 4500 5700 4500
-Wire Wire Line
-	5800 4400 5700 4400
-Wire Wire Line
-	6400 4500 6300 4500
+	5800 4550 5700 4550
+Wire Wire Line
+	5800 4450 5700 4450
+Wire Wire Line
+	5800 4350 5700 4350
+Wire Wire Line
+	6400 4450 6300 4450
 $Comp
 L power:VDC #PWR0131
 U 1 1 620A2E25
-P 5700 4400
-F 0 "#PWR0131" H 5700 4300 50  0001 C CNN
-F 1 "VDC" V 5715 4528 50  0000 L CNN
-F 2 "" H 5700 4400 50  0001 C CNN
-F 3 "" H 5700 4400 50  0001 C CNN
-	1    5700 4400
+P 5700 4350
+F 0 "#PWR0131" H 5700 4250 50  0001 C CNN
+F 1 "VDC" V 5715 4478 50  0000 L CNN
+F 2 "" H 5700 4350 50  0001 C CNN
+F 3 "" H 5700 4350 50  0001 C CNN
+	1    5700 4350
 	0    -1   -1   0
 $EndComp
@@
 L power:+12V #PWR0132
 U 1 1 620A2E2B
-P 5700 4500
-F 0 "#PWR0132" H 5700 4350 50  0001 C CNN
-F 1 "+12V" V 5715 4628 50  0000 L CNN
-F 2 "" H 5700 4500 50  0001 C CNN
-F 3 "" H 5700 4500 50  0001 C CNN
-	1    5700 4500
+P 5700 4450
+F 0 "#PWR0132" H 5700 4300 50  0001 C CNN
+F 1 "+12V" V 5715 4578 50  0000 L CNN
+F 2 "" H 5700 4450 50  0001 C CNN
+F 3 "" H 5700 4450 50  0001 C CNN
+	1    5700 4450
 	0    -1   -1   0
 $EndComp
@@
 L power:+5V #PWR0133
 U 1 1 620A2E31
-P 5700 4600
-F 0 "#PWR0133" H 5700 4450 50  0001 C CNN
-F 1 "+5V" V 5715 4728 50  0000 L CNN
-F 2 "" H 5700 4600 50  0001 C CNN
-F 3 "" H 5700 4600 50  0001 C CNN
-	1    5700 4600
-	0    -1   -1   0
-$EndComp
-Wire Wire Line
-	6300 4400 6300 4500
-Connection ~ 6300 4500
-Wire Wire Line
-	6300 4500 6300 4600
+P 5700 4550
+F 0 "#PWR0133" H 5700 4400 50  0001 C CNN
+F 1 "+5V" V 5715 4678 50  0000 L CNN
+F 2 "" H 5700 4550 50  0001 C CNN
+F 3 "" H 5700 4550 50  0001 C CNN
+	1    5700 4550
+	0    -1   -1   0
+$EndComp
+Wire Wire Line
+	6300 4350 6300 4450
+Connection ~ 6300 4450
+Wire Wire Line
+	6300 4450 6300 4550
 $Comp
 L Connector_Generic:Conn_02x03_Odd_Even J12
 U 1 1 61A78792
-P 6000 4500
-F 0 "J12" H 6450 4650 50  0000 C CNN
-F 1 "LED_V" H 6500 4750 50  0000 C CNN
-F 2 "ToolChanger:PinHeader_2x03_P1.27mm_Vertical" H 6000 4500 50  0001 C CNN
-F 3 "~" H 6000 4500 50  0001 C CNN
-	1    6000 4500
+P 6000 4450
+F 0 "J12" H 6450 4600 50  0000 C CNN
+F 1 "LED_V" H 6500 4700 50  0000 C CNN
+F 2 "ToolChanger:PinHeader_2x03_P1.27mm_Vertical" H 6000 4450 50  0001 C CNN
+F 3 "~" H 6000 4450 50  0001 C CNN
+	1    6000 4450
 	1    0    0    -1
 $EndComp
@@
 Wire Wire Line
 	4100 4500 4450 4500
+$Comp
+L ToolChanger:MillMax_004 J3
+U 1 1 6144A490
+P 2000 1425
+F 0 "J3" H 2180 1706 50  0000 L CNN
+F 1 "MillMax_004" H 2180 1615 50  0000 L CNN
+F 2 "ToolChanger:MillMax-858-10-004-10-012000" H 2270 1315 50  0001 C CNN
+F 3 "https://www.mouser.de/datasheet/2/273/MMMC_S_A0006083300_1-2558511.pdf" H 2270 1315 50  0001 C CNN
+F 4 "575-8582200480012101" H 2000 1425 50  0001 C CNN "Mouser"
+	1    2000 1425
+	1    0    0    -1
+$EndComp
+$Comp
+L ToolChanger:MillMax_004 J4
+U 1 1 61450233
+P 2000 2675
+F 0 "J4" H 2180 2956 50  0000 L CNN
+F 1 "MillMax_004" H 2180 2865 50  0000 L CNN
+F 2 "ToolChanger:MillMax-858-10-004-10-012000" H 2270 2565 50  0001 C CNN
+F 3 "https://www.mouser.de/datasheet/2/273/MMMC_S_A0006083300_1-2558511.pdf" H 2270 2565 50  0001 C CNN
+F 4 "575-8582200480012101" H 2000 2675 50  0001 C CNN "Mouser"
+	1    2000 2675
+	1    0    0    -1
+$EndComp
+Wire Wire Line
+	1750 1350 1400 1350
+NoConn ~ 1400 2900
+Text Notes -400 2950 0    50   ~ 0
+Maybe add boot pin for reflashing ability?
+$Comp
+L Connector_Generic:Conn_02x03_Odd_Even J1
+U 1 1 618086B2
+P 8250 4100
+F 0 "J1" H 8000 4500 50  0000 C CNN
+F 1 "DEBUG" H 8000 4400 50  0000 C CNN
+F 2 "ToolChanger:PinHeader_2x03_P1.27mm_Vertical" H 8250 4100 50  0001 C CNN
+F 3 "~" H 8250 4100 50  0001 C CNN
+	1    8250 4100
+	-1   0    0    1
+$EndComp
+$Comp
+L power:GND #PWR0120
+U 1 1 61BCE37C
+P 1400 3800
+F 0 "#PWR0120" H 1400 3550 50  0001 C CNN
+F 1 "GND" V 1405 3672 50  0000 R CNN
+F 2 "" H 1400 3800 50  0001 C CNN
+F 3 "" H 1400 3800 50  0001 C CNN
+	1    1400 3800
+	0    1    1    0
+$EndComp
 $EndSCHEMATC
