File: PCB/VORTAC/KiCAD/VORTAC/VORTAC_Backup.kicad_pcb (KiCad board)
At the start: 4 copper layers, 46 x 52.4 mm, 125 parts, among them IC1 TMC2209-LA, J1 DEBUG, J10 FAN_01_V, J11 FAN_02_V, J12 LED_V, J13 THERM_R, J14 918-418K2023S40001, J15 STEPPER, J16 IO, J2 Molex Micro Fit 3.0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

Commit message: More Routing
Parts:
- added D6: LED_Small, LED_SMD:LED_0402_1005Metric, F.Cu at (84.8, 102.4)
- added D7: NeoPixel_THT, LED_SMD:LED_Cree-PLCC4_2x2mm_CW, F.Cu at (100.0, 95.3)
- added D8: SK6812, LED_SMD:LED_SK6812_PLCC4_5.0x5.0mm_P3.2mm, F.Cu at (112.5, 134.2)
- added R38: R_Small, Resistor_SMD:R_0402_1005Metric, F.Cu at (84.8, 101.5)
- IC1: footprint ToolChanger:tmc_2209_package -> ToolChanger:tmc_2209_ThermalPad
- J1, J10, J11, J12: footprint Connector_PinHeader_1.27mm:PinHeader_2x03_P1.27mm_Vertical -> ToolChanger:PinHeader_2x03_P1.27mm_Vertical
- J13: footprint Connector_PinHeader_1.27mm:PinHeader_2x02_P1.27mm_Vertical -> ToolChanger:PinHeader_2x02_P1.27mm_Vertical
- J9: footprint Connector_JST:JST_PH_B2B-PH-K_1x02_P2.00mm_Vertical -> Connector_JST:JST_PH_B3B-PH-K_1x03_P2.00mm_Vertical
- moved L3 29.4 mm to (84.6, 99.0), turned to 90 degrees
- moved R35 14.9 mm to (104.2, 104.0), turned to 180 degrees
- moved R36 14.2 mm to (104.2, 103.0), turned to 180 degrees
- moved J1 7.74 mm to (87.5, 108.2)
- moved C13 4.26 mm to (93.0, 129.1)
- moved C14 4.26 mm to (101.6, 129.1)
- moved C9 4.26 mm to (97.3, 129.1)
- moved R22 4.26 mm to (95.0, 128.3)
- moved R23 4.26 mm to (103.6, 128.3)
- moved C11 4.26 mm to (105.9, 129.1)
- moved C10 4.14 mm to (93.0, 127.5)
- moved C12 4.04 mm to (101.6, 127.3)
- moved R8 3.79 mm to (82.5, 111.0), turned to 180 degrees
- moved R10 3.60 mm to (82.5, 86.9), turned to 180 degrees
- moved C16 3.33 mm to (110.5, 109.1), turned to 0 degrees
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Connections:
- net ADXL_SDO renamed Net-(U5-Pad12)
- net USART_1_RX renamed Net-(U2-Pad31)
- net USART_1_TX renamed Net-(U2-Pad30)
- J1 pad 1: DEBUG_SWCLK -> BOOT_1
- J1 pad 2: DEBUG_SWDIO -> +3V3
- J1 pad 3: GND -> NRST
- J1 pad 4: NRST -> GND
- J1 pad 5: +3V3 -> DEBUG_SWDIO
- J1 pad 6: BOOT_1 -> DEBUG_SWCLK
- J10 pad 1: FAN_1_V_OUT -> VDC
- J10 pad 2: VDC -> FAN_1_V_OUT
- J10 pad 3: FAN_1_V_OUT -> +12V
- J10 pad 4: +12V -> FAN_1_V_OUT
- J10 pad 5: FAN_1_V_OUT -> +5V
- J10 pad 6: +5V -> FAN_1_V_OUT
- J11 pad 1: FAN_2_V_OUT -> VDC
- J11 pad 2: VDC -> FAN_2_V_OUT
- J11 pad 3: FAN_2_V_OUT -> +12V
- J11 pad 4: +12V -> FAN_2_V_OUT
- J11 pad 5: FAN_2_V_OUT -> +5V
- J11 pad 6: +5V -> FAN_2_V_OUT
- J12 pad 1: LED_1_V_OUT -> VDC
- J12 pad 2: VDC -> LED_1_V_OUT
- J12 pad 3: LED_1_V_OUT -> +12V
- J12 pad 4: +12V -> LED_1_V_OUT
- J12 pad 5: LED_1_V_OUT -> +5V
- J12 pad 6: +5V -> LED_1_V_OUT
- J16 pad 3: IO_1_OUT -> IO_3_OUT
- J16 pad 5: IO_3_OUT -> IO_1_OUT
- J2 pad 1: GND -> DOCK_GND
- J2 pad 2: DOCK_GND -> DOCK_VDC
- J2 pad 3: DOCK_VDC -> GND
- J3 pad 1: TOOL_ID -> GND
- J3 pad 2: Net-(J3-Pad2) -> GND
- J3 pad 4: GND -> TOOL_DATA_H
- J4 pad 1: HOST_USB_D- -> GND
- J4 pad 2: HOST_USB_D+ -> HOST_USB_D-
- J4 pad 3: TOOL_DATA_H -> HOST_USB_D+
- J4 pad 4: TOOL_DATA_L -> TOOL_ID
- U2 pad 10: Net-(U2-Pad10) -> TOOL_ID
- U2 pad 11: Net-(U2-Pad11) -> TMC_ENN
- U2 pad 12: USART_2_TX -> TMC_UART_TX
- U2 pad 13: USART_2_RX -> TMC_UART_RX
- U2 pad 14: Net-(U2-Pad14) -> FAN_1_GATE
- U2 pad 15: Net-(U2-Pad15) -> FAN_2_GATE
- U2 pad 16: Net-(U2-Pad16) -> FAN_2_TACHO
- U2 pad 17: Net-(U2-Pad17) -> FAN_1_TACHO
- U2 pad 18: Net-(U2-Pad18) -> LED_1_PWM
- U2 pad 2: Net-(U2-Pad2) -> TMC_STEP
- U2 pad 20: Net-(U2-Pad20) -> LED_0
- U2 pad 21: USART_3_TX -> ADXL_SCL
- U2 pad 22: USART_3_RX -> ADXL_SDA
- U2 pad 25: Net-(U2-Pad25) -> ADXL_CS
- U2 pad 26: Net-(U2-Pad26) -> ADXL_INT1
- U2 pad 27: Net-(U2-Pad27) -> LED_1_GATE
- U2 pad 28: Net-(U2-Pad28) -> HOST_USB_GATE
- U2 pad 3: Net-(U2-Pad3) -> TMC_DIR
- U2 pad 38: Net-(U2-Pad38) -> THERM_1_PIN
- U2 pad 39: DEBUG_SWO -> IO_3_OUT
- U2 pad 4: Net-(U2-Pad4) -> TMC_DIAG
- U2 pad 40: Net-(U2-Pad40) -> IO_2_OUT
- U2 pad 41: Net-(U2-Pad41) -> IO_1_OUT
- U2 pad 42: Net-(U2-Pad42) -> HEATER_GATE
- U5 pad 13: ADXL_SDI -> ADXL_SDA
Routing:
- net TOOL_ID: track 7.26 -> 45.8 mm
- net HOST_USB_D+: track 0.00 -> 28.8 mm
- net HOST_USB_D-: track 0.00 -> 23.0 mm
- net TOOL_DATA_L: track 3.32 -> 20.8 mm
- net TOOL_DATA_H: track 6.56 -> 23.9 mm
- net FAN_2_GATE: track 0.00 -> 17.1 mm
- net DOCK_GND: track 2.20 -> 18.3 mm, vias 12 -> 24
- net Net-(D3-Pad2): track 1.21 -> 16.4 mm, vias 0 -> 2
- net FAN_1_GATE: track 0.00 -> 14.8 mm
- net +5V: track 0.00 -> 14.5 mm, vias 0 -> 3
- net VDC: track 7.50 -> 21.2 mm, vias 22 -> 23
- net GND: track 33.5 -> 44.8 mm, vias 36 -> 39
- net DOCK_VDC: track 2.22 -> 12.5 mm, vias 12 -> 23
- net LED_1_PWM: track 0.00 -> 9.70 mm
- net FAN_2_V_OUT: track 0.00 -> 8.70 mm
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- added copper zone on B.Cu, net DOCK_GND
- added copper zone on B.Cu, net DOCK_VDC
- added copper zone on B.Cu, net HEATER_DRAIN
- removed copper zone on In1.Cu, net DOCK_GND
Other:
- net class 0.35mm added: clearance 0.2, trace_width 0.35, via_dia 0.8, via_drill 0.4
- net class 0.5mm added: clearance 0.2, trace_width 0.5, via_dia 1.2, via_drill 0.6
- net class 2.0mm added: clearance 0.2, trace_width 2, via_dia 0.8, via_drill 0.4
- net class Wide removed
