File: PCB/VORTAC/KiCAD/VORTAC_REV1/MCU.kicad_sch (KiCad schematic)
At the start: 34 parts, among them IC1 TMC2209-LA, U2 STM32F103C8Tx, U6 SN65HVD232DR

Commit message: hallo
Parts:
- removed D7: NeoPixel_THT, LED_SMD:LED_Cree-PLCC4_2x2mm_CW, symbol LED:NeoPixel_THT
- added U5: STM32G0B1C_B-C-E_Tx, Package_QFP:LQFP-48_7x7mm_P0.5mm, symbol MCU_ST_STM32G0:STM32G0B1C_B-C-E_Tx
- IC1: footprint ToolChanger:tmc_2209_ThermalPad -> ToolChanger:tmc_2209_package
Connections:
- net ADXL_CS: no longer names the net of U2.14 (PA4)
- net ADXL_INT1: no longer names the net of U2.13 (PA3)
- net ADXL_SCL: no longer names the net of U2.15 (PA5)
- net ADXL_SDI: no longer names the net of U2.17 (PA7)
- net ADXL_SDO: no longer names the net of U2.16 (PA6)
- net FAN_1_GATE: no longer names the net of U2.42 (PB6)
- net FAN_2_GATE: no longer names the net of U2.43 (PB7)
- net HEATER_GATE: no longer names the net of U2.27 (PB14)
- net HOST_USB_GATE: no longer names the net of U2.10 (PA0)
- net IO_1_OUT_PIN: no longer names the net of U2.26 (PB13)
- net IO_2_OUT_PIN: no longer names the net of U2.25 (PB12)
- net IO_3_OUT_PIN: no longer names the net of U2.22 (PB11)
- net LED_1_GATE: no longer names the net of U2.11 (PA1)
- net THERM_1_PIN: no longer names the net of U2.21 (PB10)
Other:
- note removed: "this interrupt should be obsolete??"

Commit message: yipppieee
Parts:
- removed R31: 1K, Resistor_SMD:R_0402_1005Metric, symbol Device:R_Small
- removed U5: STM32G0B1C_B-C-E_Tx, Package_QFP:LQFP-48_7x7mm_P0.5mm, symbol MCU_ST_STM32G0:STM32G0B1C_B-C-E_Tx
- added C1, C4, C6, C9: 470pF 100V, Capacitor_SMD:C_0603_1608Metric, symbol Device:C_Small
- added C10, C2: 0.1uF 50V, Capacitor_SMD:C_0603_1608Metric, symbol Device:C_Small
- added JP1: Jumper, Connector_PinHeader_1.27mm:PinHeader_2x01_P1.27mm_Vertical, symbol Jumper:Jumper_2_Small_Open
- added L1: Common Choke, Inductor_SMD:L_CommonModeChoke_Coilcraft_0805USB, symbol Filter:Choke_Wurth_WE-CNSW_744232090
- added R10: 120R, Resistor_SMD:R_0402_1005Metric, symbol Device:R_Small
- added R9: 100R, Resistor_SMD:R_0402_1005Metric, symbol Device:R_Small
- C22: value 0.1uF 50V -> 4.7uF 50V
- C34: footprint Capacitor_SMD:CP_Elec_8x6.9 -> Capacitor_SMD:CP_Elec_6.3x7.7; LCSC (none) -> C2983388
- R30, R34: value 0.1R 1% -> 0.22R 1%
- R32, R33: value 22K -> 10K
Connections:
- net TMC_UART_TX is gone; now on net TMC_UART: U2.30 (PA9)
- net +3V3: now also R33.2
- net CAN_H: now also L1.2, R10.1; no longer U6.7 (CANH)
- net CAN_L: now also JP1.2 (B), L1.3; no longer U6.6 (CANL)
- net ENDSTOP_X: now also U2.11 (PA1)
- net ENDSTOP_Z: now also U2.10 (PA0)
- net GND: now also C1.2, C10.2, C2.2, C4.2, C6.2, C9.2; no longer R33.2
- net STEP_1_A1: now also C4.1
- net STEP_1_A2: now also C1.1
- net STEP_1_B1: now also C6.1
- net STEP_1_B2: now also C9.1
- net TMC_BRA: now also C10.1
- net TMC_BRB: now also C2.1
- net TMC_DIAG: now also R9.2; no longer U2.38 (PA15)
- net TMC_UART_RX renamed TMC_UART
- net TMC_UART: no longer U2.31 (PA10)
- new net: R9.1, U2.38 (PA15)
- new net: L1.4, U6.6 (CANL)
- new net: L1.1, U6.7 (CANH)
- new net: JP1.1 (A), R10.2
Other:
- note added: "goes nowhere???"
- moved on the sheet: C35, R33, R35, R36, U2

Commit message: Wayollaaaaa
Parts:
- added C13: 0.1uF 50V, Capacitor_SMD:C_0603_1608Metric, symbol Device:C_Small
- added R11, R12: 10K, Resistor_SMD:R_0402_1005Metric, symbol Device:R_Small
- added SW1: Boot, symbol Switch:SW_Push
- added SW2: Reset, symbol Switch:SW_Push
- HSE1: LCSC C518155 -> C5261255
- U2: value STM32F103C8Tx -> STM32F103C8T6
Connections:
- net +3V3: now also SW1.2
- net BOOT_0: now also R11.1, SW1.1
- net BOOT_1: now also R12.1
- net GND: now also C13.2, R11.2, R12.2, SW2.2
- net NRST: now also C13.1, SW2.1
Other:
- note added: "BOOT_1 needed for System Memory boot (bootloader) needs pull down resistor"
- note added: "BOOT_1 optional for SRAM boot needs pull down resistor"
- note added: "Caps and Res undefined"
- note added: "MCU"
- note added: "MCU Peripherals"
- note added: "MCU Power and Timing"
- note added: "Optional Asynchronous SW??"
- note removed: "BOOT 1 needs pulldown"
- note removed: "Optional Asynchronous SW"
- note removed: "SDO is adress?? DO we need that???"
- note removed: "goes nowhere???"
- moved on the sheet: C33, C35, C36, C37, C38, C39, C40, C42, C43, C44, C45, D6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

Commit message: Fixed Library stuff
Parts:
- IC1: footprint ToolChanger:tmc_2209_package -> Vortac:tmc_2209_package
- L1: footprint Inductor_SMD:L_CommonModeChoke_Coilcraft_0805USB -> Vortac:L_CommonModeChoke_Coilcraft_0805USB
- SW1, SW2: footprint (none) -> Vortac:KEY-SMD_B3U-1000PM; LCSC C720477 -> C231329
Changed lines of the file:
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@@
 			)
 		)
-		(property "Footprint" "ToolChanger:tmc_2209_package"
+		(property "Footprint" "Vortac:tmc_2209_package"
 			(at 212.09 69.85 90)
 			(effects
@@
 			)
 		)
-		(property "Footprint" ""
+		(property "Footprint" "Vortac:KEY-SMD_B3U-1000PM"
 			(at 115.57 171.45 0)
 			(effects
@@
 			)
 		)
-		(property "Datasheet" "https://www.lcsc.com/datasheet/lcsc_datasheet_2504101957_XUNPU-TS-1088-AR02016_C720477.pdf"
+		(property "Datasheet" "https://www.lcsc.com/datasheet/lcsc_datasheet_2504101957_Omron-Electronics-B3U-1000P_C231329.pdf"
 			(at 115.57 171.45 0)
 			(effects
@@
 			)
 		)
-		(property "LCSC" "C720477"
+		(property "LCSC" "C231329"
 			(at 115.57 176.53 0)
 			(effects
@@
 			)
 		)
-		(property "Footprint" "Inductor_SMD:L_CommonModeChoke_Coilcraft_0805USB"
+		(property "Footprint" "Vortac:L_CommonModeChoke_Coilcraft_0805USB"
 			(at 201.93 148.59 0)
 			(effects
@@
 			)
 		)
-		(property "Footprint" ""
+		(property "Footprint" "Vortac:KEY-SMD_B3U-1000PM"
 			(at 115.57 154.94 0)
 			(effects
@@
 			)
 		)
-		(property "Datasheet" "https://www.lcsc.com/datasheet/lcsc_datasheet_2504101957_XUNPU-TS-1088-AR02016_C720477.pdf"
+		(property "Datasheet" "https://www.lcsc.com/datasheet/lcsc_datasheet_2504101957_Omron-Electronics-B3U-1000P_C231329.pdf"
 			(at 115.57 154.94 0)
 			(effects
@@
 			)
 		)
-		(property "LCSC" "C720477"
+		(property "LCSC" "C231329"
 			(at 115.57 160.02 0)
 			(effects

Commit message: Kanoolaaaa
Parts:
- removed R37: R_Small, Resistor_SMD:R_0402_1005Metric, symbol Device:R_Small
- removed U6: SN65HVD232DR, Package_SO:SOIC-8_3.9x4.9mm_P1.27mm, symbol ToolChanger:SN65HVD232DR
- added U8: TJA1044GTK/3Z, Vortac:HVSON-8-1EP_3x3mm_P0.65mm_EP1.6x2.4mm, symbol Vortac:TJA1044GTK_3Z
- C42, C43: value C_Small -> 16pF
Connections:
- net GND1 is gone; now on net GND: C42.2, C43.2, HSE1.2, HSE1.4
- net +3V3: now also U8.5 (VIO); no longer C33.2, C35.1
- net CAN_RX: now also U8.4 (RXD)
- net CAN_TX: now also U8.1 (TXD)
- net GND: now also U8.2 (GND), U8.8 (STB), U8.9 (EP)
- net HSE_OSC_OUT: now also C43.1, HSE1.3
- net at L1.4: now also U8.6 (CANL)
- net at L1.1: now also U8.7 (CANH)
- new net +5V: U8.3 (VCC)
Other:
- note added: "Caps could also be 15pF (closest standard value)"
- note added: "OLD Canbus transciever used a filtering Cap on VCC +3.3 Check if this is still needed"
- note removed: "Caps and Res undefined"
- moved on the sheet: C35, C36, C37, C38, C39, C40, C42, C43, C44, C45, HSE1, JP1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

Commit message: Liebe Griasse zurrueck
Parts:
- added C17: 0.1uF 16V, Capacitor_SMD:C_0402_1005Metric, symbol Device:C_Small
- D6: LCSC (none) -> C130724
- R38: value R_Small -> 22R
Connections:
- net +3.3VA: no longer U2.9 (VDDA)
- net +3V3: now also C33.2, C35.1, U2.9 (VDDA)
- net +5V: now also C17.1
- net DEBUG_SWO: now also U2.39 (PB3)
- net GND: now also C17.2
- net TMC_ENN: no longer U2.40 (PB4)
- net AS_NCS: now reaches U2.14 (PA4)
- net AS_CLK: now reaches U2.15 (PA5)
- net AS_MISO: now reaches U2.16 (PA6)
- net AS_MOSI: now reaches U2.17 (PA7)
Other:
- note added: "Inline Resistor USB??"
- note added: "Removed Analog Refference Voltage Filter"
- note removed: "OLD Canbus transciever used a filtering Cap on VCC +3.3 Check if this is still needed"
- moved on the sheet: C33, C35, C44, C45, L3
