File: PCB/VORTAC/KiCAD/VORTAC_REV1/MCU.kicad_sch (KiCad schematic)
At the start: 44 parts, among them IC1 TMC2209-LA, SW1 Boot, SW2 Reset, U2 STM32F103C8T6, U8 TJA1044GTK/3Z, Y1 8MHz

Commit message: BOMBOM
Other:
- note added: "PA9-10 can be used to connect a USB to Serial adapter to USART1 for USB Flashing without USB Bootloader"
Changed lines of the file:
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@@
+		)
+	)
+	(text "PA9-10 can be used to connect a USB to Serial\nadapter to USART1 for USB Flashing without USB Bootloader"
+		(exclude_from_sim no)
+		(at 100.838 85.852 0)
+		(effects
+			(font
+				(size 0.7874 0.7874)
+			)
+			(justify left top)
 		)
 	)

Commit message: Anned Parts
Parts:
- C1, C4, C6, C9: LCSC C1591 -> C326973; description (none) -> NP0 better than X7R
- C10, C13, C2, C21, C24, C26, C29: footprint Capacitor_SMD:C_0603_1608Metric -> Capacitor_SMD:C_0402_1005Metric; LCSC C1591 -> C5182432
- C17, C35: value 0.1uF 16V -> 0.1uF 50V; LCSC (none) -> C5182432
- C22: LCSC C1591 -> C513577
- C23: value 22nF X7R 10% 50V -> 22nF 50V; footprint Capacitor_SMD:C_0603_1608Metric -> Capacitor_SMD:C_0402_1005Metric; LCSC (none) -> C107026; description (none) -> 50V 10% X7R
- C33, C36, C37, C38, C39: value 0.1uF 16V -> 0.1uF 50V; LCSC C1525 -> C5182432
- C40: value 4.7uF 10V -> 4.7uF 50V; footprint Capacitor_SMD:C_0402_1005Metric -> Capacitor_SMD:C_0603_1608Metric; LCSC C368809 -> C513577; description (none) -> could be higher
- C42, C43: value 16pF -> 16pF 50V; LCSC (none) -> C513591; description (none) -> close to crystal
- IC1: LCSC C465949 -> C2150710
- L1: LCSC C383338 -> C3029267
- R10: value 110R -> 115R; LCSC (none) -> C295872; description (none) -> hard to calculate make jumpable 120 Ohm ?
- R11, R12, R32, R9: LCSC (none) -> C60490
- R13: LCSC (none) -> C106235
- R30, R34: description (none) -> TODO evaluate Motor Current
- R7: value 100R -> 115R; LCSC (none) -> C295872
- U8: footprint Vortac:HVSON-8-1EP_3x3mm_P0.65mm_EP1.6x2.4mm -> Vortac:HVSON-8_L3.0-W3.0-P0.65-BL-EP; LCSC (none) -> C2157795; LCSC Part C2157795 -> (none)
Other:
- note removed: "PA9-10 can be used to connect a USB to Serial adapter to USART1 for USB Flashing without USB Bootloader"

Commit message: Evil Mita is v00:98
Parts:
- C1, C4, C6, C9: description NP0 better than X7R -> (none); notes (none) -> NP0 better than X7R
- C23: description 50V 10% X7R -> (none); notes (none) -> 50V 10% X7R
- C40: description could be higher -> (none); notes (none) -> could be higher
- C42, C43: description close to crystal -> (none); notes (none) -> close to crystal
- R10: description hard to calculate make jumpable 120 Ohm ? -> (none); notes (none) -> hard to calculate make jumpable 120 Ohm ?
- R30, R34: footprint Resistor_SMD:R_1206_3216Metric -> Resistor_SMD:R_0805_2012Metric; description TODO evaluate Motor Current -> (none); notes (none) -> TODO evaluate Motor Current

Commit message: No Body knows.... The trouble I've seen
Connections:
- net CAN_H: now also L1.3, R10.1; no longer L1.2
- net CAN_L: now also L1.2; no longer L1.3, R10.1
- net at U8.6 (CANL): now also L1.1; no longer L1.4
- net at U8.7 (CANH): now also L1.4; no longer L1.1
- net CAN_TRM_L renamed CAN_TRM_H
Other:
- moved on the sheet: L1, R10
Changed lines of the file:
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@@
 	)
 	(junction
-		(at 243.84 137.16)
+		(at 251.46 133.35)
 		(diameter 0)
 		(color 0 0 0 0)
@@
 	)
 	(junction
-		(at 248.92 132.08)
+		(at 256.54 128.27)
 		(diameter 0)
 		(color 0 0 0 0)
@@
 	(wire
 		(pts
-			(xy 223.52 132.08) (xy 223.52 133.35)
-		)
-		(stroke
-			(width 0)
-			(type default)
-		)
-	)
-	(wire
-		(pts
 			(xy 173.99 147.32) (xy 173.99 149.86)
 		)
@@
 	(wire
 		(pts
-			(xy 243.84 137.16) (xy 255.27 137.16)
+			(xy 251.46 133.35) (xy 262.89 133.35)
 		)
 		(stroke
@@
 	(wire
 		(pts
-			(xy 226.06 132.08) (xy 223.52 132.08)
-		)
-		(stroke
-			(width 0)
-			(type default)
-		)
-	)
-	(wire
-		(pts
 			(xy 54.61 90.17) (xy 59.69 90.17)
 		)
@@
 	(wire
 		(pts
-			(xy 236.22 137.16) (xy 243.84 137.16)
+			(xy 243.84 133.35) (xy 251.46 133.35)
 		)
 		(stroke
@@
 	(wire
 		(pts
+			(xy 228.6 135.89) (xy 210.82 135.89)
+		)
+		(stroke
+			(width 0)
+			(type default)
+		)
+	)
+	(wire
+		(pts
 			(xy 168.91 30.48) (xy 173.99 30.48)
 		)
@@
 	(wire
 		(pts
-			(xy 226.06 137.16) (xy 223.52 137.16)
-		)
-		(stroke
-			(width 0)
-			(type default)
-		)
-	)
-	(wire
-		(pts
 			(xy 44.45 182.88) (xy 48.26 182.88)
 		)
@@
 	(wire
 		(pts
-			(xy 210.82 135.89) (xy 223.52 135.89)
+			(xy 228.6 128.27) (xy 233.68 128.27)
 		)
 		(stroke
@@
 	(wire
 		(pts
-			(xy 223.52 137.16) (xy 223.52 135.89)
-		)
-		(stroke
-			(width 0)
-			(type default)
-		)
-	)
-	(wire
-		(pts
 			(xy 44.45 172.72) (xy 48.26 172.72)
 		)
@@
 	(wire
 		(pts
+			(xy 228.6 128.27) (xy 228.6 135.89)
+		)
+		(stroke
+			(width 0)
+			(type default)
+		)
+	)
+	(wire
+		(pts
 			(xy 269.24 40.64) (xy 261.62 40.64)
 		)
@@
 	(wire
 		(pts
-			(xy 223.52 133.35) (xy 210.82 133.35)
+			(xy 210.82 133.35) (xy 233.68 133.35)
 		)
 		(stroke
@@
 	(wire
 		(pts
-			(xy 236.22 132.08) (xy 248.92 132.08)
+			(xy 243.84 128.27) (xy 256.54 128.27)
 		)
 		(stroke
@@
 	(wire
 		(pts
-			(xy 243.84 149.86) (xy 255.27 149.86)
+			(xy 251.46 146.05) (xy 262.89 146.05)
 		)
 		(stroke
@@
 	(wire
 		(pts
-			(xy 243.84 137.16) (xy 243.84 140.97)
+			(xy 251.46 133.35) (xy 251.46 137.16)
 		)
 		(stroke
@@
 	(wire
 		(pts
-			(xy 248.92 132.08) (xy 255.27 132.08)
+			(xy 256.54 128.27) (xy 262.89 128.27)
 		)
 		(stroke
@@
 	(wire
 		(pts
-			(xy 243.84 146.05) (xy 243.84 149.86)
+			(xy 251.46 142.24) (xy 251.46 146.05)
 		)
 		(stroke
@@
 	(wire
 		(pts
-			(xy 248.92 132.08) (xy 248.92 144.78)
+			(xy 256.54 128.27) (xy 256.54 140.97)
 		)
 		(stroke
@@
 	(wire
 		(pts
-			(xy 248.92 144.78) (xy 255.27 144.78)
+			(xy 256.54 140.97) (xy 262.89 140.97)
 		)
 		(stroke
@@
 	(global_label "CAN_H"
 		(shape input)
-		(at 255.27 132.08 0)
+		(at 262.89 133.35 0)
 		(effects
 			(font
@@
 		)
 		(property "Intersheetrefs" "${INTERSHEET_REFS}"
-			(at 255.27 132.08 0)
+			(at 262.89 133.35 0)
 			(effects
 				(font
@@
 	(global_label "CAN_L"
 		(shape input)
-		(at 255.27 137.16 0)
+		(at 262.89 128.27 0)
 		(effects
 			(font
@@
 		)
 		(property "Intersheetrefs" "${INTERSHEET_REFS}"
-			(at 255.27 137.16 0)
+			(at 262.89 128.27 0)
 			(effects
 				(font
@@
 	(global_label "CAN_TRM_L"
 		(shape input)
-		(at 255.27 149.86 0)
+		(at 262.89 140.97 0)
 		(effects
 			(font
@@
 		)
 		(property "Intersheetrefs" "${INTERSHEET_REFS}"
-			(at 255.27 149.86 0)
+			(at 262.89 140.97 0)
 			(effects
 				(font
@@
 	(global_label "CAN_TRM_H"
 		(shape input)
-		(at 255.27 144.78 0)
+		(at 262.89 146.05 0)
 		(effects
 			(font
@@
 		)
 		(property "Intersheetrefs" "${INTERSHEET_REFS}"
-			(at 255.27 144.78 0)
+			(at 262.89 146.05 0)
 			(effects
 				(font
@@
 	(symbol
 		(lib_id "Filter:Choke_Wurth_WE-CNSW_744232090")
-		(at 231.14 134.62 0)
+		(at 238.76 130.81 0)
 		(unit 1)
 		(exclude_from_sim no)
@@
 		(dnp no)
 		(property "Reference" "L1"
-			(at 230.886 130.556 0)
+			(at 238.506 126.746 0)
 			(effects
 				(font
@@
 		)
 		(property "Value" "Common Choke"
-			(at 231.902 138.684 0)
+			(at 239.522 134.874 0)
 			(effects
 				(font
@@
 		)
 		(property "Footprint" "Vortac:L_CommonModeChoke_Coilcraft_0805USB"
-			(at 231.14 144.78 0)
+			(at 238.76 140.97 0)
 			(effects
 				(font
@@
 		)
 		(property "Datasheet" "https://www.lcsc.com/datasheet/lcsc_datasheet_2412201235_TDK-ACM2012-201-2P-T001_C383338.pdf"
-			(at 231.14 142.24 0)
+			(at 238.76 138.43 0)
 			(effects
 				(font
@@
 		)
 		(property "Description" ""
-			(at 231.14 134.62 0)
+			(at 238.76 130.81 0)
 			(effects
 				(font
@@
 		)
 		(property "LCSC" "C3029267"
-			(at 231.14 134.62 0)
+			(at 238.76 130.81 0)
 			(effects
 				(font
@@
 	(symbol
 		(lib_id "Device:R_Small")
-		(at 243.84 143.51 0)
+		(at 251.46 139.7 0)
 		(unit 1)
 		(exclude_from_sim no)
@@
 		(dnp no)
 		(property "Reference" "R10"
-			(at 246.126 148.844 90)
+			(at 253.746 145.034 90)
 			(effects
 				(font
@@
 		)
 		(property "Value" "115R"
-			(at 246.126 144.272 90)
+			(at 253.746 140.462 90)
 			(effects
 				(font
@@
 		)
 		(property "Footprint" "Resistor_SMD:R_0402_1005Metric"
-			(at 243.84 143.51 0)
+			(at 251.46 139.7 0)
 			(effects
 				(font
@@
 		)
 		(property "Datasheet" "~"
-			(at 243.84 143.51 0)
+			(at 251.46 139.7 0)
 			(effects
 				(font
@@
 		)
 		(property "Description" "Resistor, small symbol"
-			(at 243.84 143.51 0)
+			(at 251.46 139.7 0)
 			(effects
 				(font
@@
 		)
 		(property "LCSC" "C295872"
-			(at 243.84 143.51 0)
+			(at 251.46 139.7 0)
 			(effects
 				(font
@@
 		)
 		(property "notes" "hard to calculate make jumpable 120 Ohm ? "
-			(at 243.84 143.51 0)
+			(at 251.46 139.7 0)
 			(effects
 				(font

Commit message: Route me like one of you French girls
Connections:
- net CAN_TRM_H is gone; now on net CAN_L: R10.2
- net CAN_TRM: no longer names the net of U2.42 (PB6)
- no-connect marks 15 -> 16
Changed lines of the file:
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@@
 		(at 54.61 80.01)
 	)
+	(no_connect
+		(at 54.61 77.47)
+	)
 	(wire
 		(pts
@@
 	(wire
 		(pts
+			(xy 251.46 146.05) (xy 256.54 146.05)
+		)
+		(stroke
+			(width 0)
+			(type default)
+		)
+	)
+	(wire
+		(pts
 			(xy 39.37 138.43) (xy 39.37 132.08)
 		)
@@
 	(wire
 		(pts
-			(xy 40.64 77.47) (xy 59.69 77.47)
+			(xy 54.61 77.47) (xy 59.69 77.47)
 		)
 		(stroke
@@
 	(wire
 		(pts
+			(xy 256.54 128.27) (xy 256.54 146.05)
+		)
+		(stroke
+			(width 0)
+			(type default)
+		)
+	)
+	(wire
+		(pts
 			(xy 240.03 48.26) (xy 250.19 48.26)
 		)
@@
 	(wire
 		(pts
-			(xy 251.46 146.05) (xy 262.89 146.05)
-		)
-		(stroke
-			(width 0)
-			(type default)
-		)
-	)
-	(wire
-		(pts
 			(xy 54.61 54.61) (xy 59.69 54.61)
 		)
@@
 	(wire
 		(pts
-			(xy 256.54 128.27) (xy 256.54 140.97)
-		)
-		(stroke
-			(width 0)
-			(type default)
-		)
-	)
-	(wire
-		(pts
 			(xy 54.61 39.37) (xy 59.69 39.37)
 		)
@@
 	(wire
 		(pts
-			(xy 256.54 140.97) (xy 262.89 140.97)
-		)
-		(stroke
-			(width 0)
-			(type default)
-		)
-	)
-	(wire
-		(pts
 			(xy 118.11 148.59) (xy 127 148.59)
 		)
@@
 		(property "Intersheetrefs" "${INTERSHEET_REFS}"
 			(at 54.61 175.26 0)
-			(effects
-				(font
-					(size 1.27 1.27)
-				)
-				(hide yes)
-			)
-		)
-	)
-	(global_label "CAN_TRM_L"
-		(shape input)
-		(at 262.89 140.97 0)
-		(effects
-			(font
-				(size 1.27 1.27)
-			)
-			(justify left)
-		)
-		(property "Intersheetrefs" "${INTERSHEET_REFS}"
-			(at 262.89 140.97 0)
 			(effects
 				(font
@@
 			(effects
 				(font
-					(size 1.27 1.27)
-				)
-				(hide yes)
-			)
-		)
-	)
-	(global_label "CAN_TRM"
-		(shape input)
-		(at 40.64 77.47 180)
-		(effects
-			(font
-				(size 1.27 1.27)
-			)
-			(justify right)
-		)
-		(property "Intersheetrefs" "${INTERSHEET_REFS}"
-			(at 40.64 77.47 0)
-			(effects
-				(font
-					(size 1.27 1.27)
-				)
-				(hide yes)
-			)
-		)
-	)
-	(global_label "CAN_TRM_H"
-		(shape input)
-		(at 262.89 146.05 0)
-		(effects
-			(font
-				(size 1.27 1.27)
-			)
-			(justify left)
-		)
-		(property "Intersheetrefs" "${INTERSHEET_REFS}"
-			(at 262.89 146.05 0)
-			(effects
-				(font

Commit message: FML
Parts:
- U8: footprint Vortac:HVSON-8_L3.0-W3.0-P0.65-BL-EP -> Vortac:HVSON-8-1EP_3x3mm_P0.65mm_EP1.6x2.4mm
Connections:
- net DAMPEND_USB_DL: now reaches R35.2, U2.32 (PA11)
- net DAMPEND_USB_DH: now reaches R36.2, U2.33 (PA12)
- net CAN_L_CHOKE: now reaches L1.1, U8.6 (CANL)
- net CAN_H_CHOKE: now reaches L1.4, U8.7 (CANH)
Other:
- moved on the sheet: L1, R35, R36
Changed lines of the file:
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@@
 	(wire
 		(pts
-			(xy 102.87 90.17) (xy 111.76 90.17)
+			(xy 121.92 90.17) (xy 128.27 90.17)
 		)
 		(stroke
@@
 	(wire
 		(pts
-			(xy 92.71 90.17) (xy 97.79 90.17)
+			(xy 92.71 90.17) (xy 116.84 90.17)
 		)
 		(stroke
@@
 	(wire
 		(pts
-			(xy 243.84 133.35) (xy 251.46 133.35)
+			(xy 246.38 133.35) (xy 251.46 133.35)
 		)
 		(stroke
@@
 	(wire
 		(pts
-			(xy 228.6 135.89) (xy 210.82 135.89)
+			(xy 232.41 135.89) (xy 210.82 135.89)
 		)
 		(stroke
@@
 	(wire
 		(pts
-			(xy 228.6 128.27) (xy 233.68 128.27)
+			(xy 232.41 128.27) (xy 236.22 128.27)
 		)
 		(stroke
@@
 	(wire
 		(pts
-			(xy 228.6 128.27) (xy 228.6 135.89)
+			(xy 232.41 128.27) (xy 232.41 135.89)
 		)
 		(stroke
@@
 	(wire
 		(pts
-			(xy 210.82 133.35) (xy 233.68 133.35)
+			(xy 210.82 133.35) (xy 236.22 133.35)
 		)
 		(stroke
@@
 	(wire
 		(pts
-			(xy 243.84 128.27) (xy 256.54 128.27)
+			(xy 246.38 128.27) (xy 256.54 128.27)
 		)
 		(stroke
@@
 	(wire
 		(pts
-			(xy 92.71 92.71) (xy 101.6 92.71)
+			(xy 92.71 92.71) (xy 116.84 92.71)
 		)
 		(stroke
@@
 	(wire
 		(pts
-			(xy 106.68 92.71) (xy 111.76 92.71)
+			(xy 121.92 92.71) (xy 128.27 92.71)
 		)
 		(stroke
@@
 		)
 	)
+	(label "DAMPEND_USB_DH"
+		(at 93.98 92.71 0)
+		(effects
+			(font
+				(size 1.27 1.27)
+			)
+			(justify left bottom)
+		)
+	)
+	(label "CAN_L_CHOKE"
+		(at 215.9 135.89 0)
+		(effects
+			(font
+				(size 1.27 1.27)
+			)
+			(justify left bottom)
+		)
+	)
+	(label "CAN_H_CHOKE"
+		(at 215.9 133.35 0)
+		(effects
+			(font
+				(size 1.27 1.27)
+			)
+			(justify left bottom)
+		)
+	)
+	(label "DAMPEND_USB_DL"
+		(at 93.98 90.17 0)
+		(effects
+			(font
+				(size 1.27 1.27)
+			)
+			(justify left bottom)
+		)
+	)
 	(global_label "HSE_OSC_OUT"
 		(shape input)
@@
 	(global_label "USB_D+"
 		(shape input)
-		(at 111.76 92.71 0)
+		(at 128.27 92.71 0)
 		(effects
 			(font
@@
 		)
 		(property "Intersheetrefs" "${INTERSHEET_REFS}"
-			(at 111.76 92.71 0)
+			(at 128.27 92.71 0)
 			(effects
 				(font
@@
 	(global_label "USB_D-"
 		(shape input)
-		(at 111.76 90.17 0)
+		(at 128.27 90.17 0)
 		(effects
 			(font
@@
 		)
 		(property "Intersheetrefs" "${INTERSHEET_REFS}"
-			(at 111.76 90.17 0)
+			(at 128.27 90.17 0)
 			(effects
 				(font
@@
 	(symbol
 		(lib_id "Device:R_Small")
-		(at 100.33 90.17 270)
+		(at 119.38 90.17 270)
 		(unit 1)
 		(exclude_from_sim no)
@@
 		(dnp no)
 		(property "Reference" "R35"
-			(at 96.52 89.154 90)
+			(at 115.57 89.154 90)
 			(effects
 				(font
@@
 		)
 		(property "Value" "22R"
-			(at 104.394 89.154 90)
+			(at 123.444 89.154 90)
 			(effects
 				(font
@@
 		)
 		(property "Footprint" "Resistor_SMD:R_0402_1005Metric"
-			(at 100.33 88.392 90)
+			(at 119.38 88.392 90)
 			(effects
 				(font
@@
 		)
 		(property "Datasheet" "~"
-			(at 100.33 90.17 0)
+			(at 119.38 90.17 0)
 			(effects
 				(font
@@
 		)
 		(property "Description" "Resistor, small symbol"
-			(at 100.33 90.17 0)
+			(at 119.38 90.17 0)
 			(effects
 				(font
@@
 	(symbol
 		(lib_id "Device:R_Small")
-		(at 104.14 92.71 270)
+		(at 119.38 92.71 270)
 		(unit 1)
 		(exclude_from_sim no)
@@
 		(dnp no)
 		(property "Reference" "R36"
-			(at 100.33 91.948 90)
+			(at 115.57 91.948 90)
 			(effects
 				(font
@@
 		)
 		(property "Value" "22R"
-			(at 108.204 91.694 90)
+			(at 123.444 91.694 90)
 			(effects
 				(font
@@
 		)
 		(property "Footprint" "Resistor_SMD:R_0402_1005Metric"
-			(at 104.14 90.932 90)
+			(at 119.38 90.932 90)
 			(effects
 				(font
@@
 		)
 		(property "Datasheet" "~"
-			(at 104.14 92.71 0)
+			(at 119.38 92.71 0)
 			(effects
 				(font
@@
 		)
 		(property "Description" "Resistor, small symbol"
-			(at 104.14 92.71 0)
+			(at 119.38 92.71 0)
 			(effects
 				(font
@@
 			)
 		)
-		(property "Footprint" "Vortac:HVSON-8_L3.0-W3.0-P0.65-BL-EP"
+		(property "Footprint" "Vortac:HVSON-8-1EP_3x3mm_P0.65mm_EP1.6x2.4mm"
 			(at 200.66 146.05 0)
 			(effects
@@
 	(symbol
 		(lib_id "Filter:Choke_Wurth_WE-CNSW_744232090")
-		(at 238.76 130.81 0)
+		(at 241.3 130.81 0)
 		(unit 1)
 		(exclude_from_sim no)
@@
 		(dnp no)
 		(property "Reference" "L1"
-			(at 238.506 126.746 0)
+			(at 241.046 126.746 0)
 			(effects
 				(font
@@
 		)
 		(property "Value" "Common Choke"
-			(at 239.522 134.874 0)
+			(at 242.062 134.874 0)
 			(effects
 				(font
@@
 		)
 		(property "Footprint" "Vortac:L_CommonModeChoke_Coilcraft_0805USB"
-			(at 238.76 140.97 0)
+			(at 241.3 140.97 0)
 			(effects
 				(font
@@
 		)
 		(property "Datasheet" "https://www.lcsc.com/datasheet/lcsc_datasheet_2412201235_TDK-ACM2012-201-2P-T001_C383338.pdf"
-			(at 238.76 138.43 0)
+			(at 241.3 138.43 0)
 			(effects
 				(font
@@
 		)
 		(property "Description" ""
-			(at 238.76 130.81 0)
+			(at 241.3 130.81 0)
 			(effects
 				(font
@@
 		)
 		(property "LCSC" "C3029267"
-			(at 238.76 130.81 0)
+			(at 241.3 130.81 0)
 			(effects
 				(font

Commit message: USB C Pain
Connections:
- net DAMPEND_USB_DH renamed DAMPEND_USB_D+
- net DAMPEND_USB_DL renamed DAMPEND_USB_D-
Changed lines of the file:
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@@
 		)
 	)
-	(label "DAMPEND_USB_DH"
+	(label "DAMPEND_USB_D+"
 		(at 93.98 92.71 0)
 		(effects
@@
 		)
 	)
-	(label "DAMPEND_USB_DL"
+	(label "DAMPEND_USB_D-"
 		(at 93.98 90.17 0)
 		(effects

Commit message: KONGSTRONG
Parts:
- R30, R34: value 0.22R 1% -> 0.68R 1%; LCSC C346768 -> C912570
Changed lines of the file:
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@@
 			)
 		)
-		(property "Value" "0.22R 1%"
+		(property "Value" "0.68R 1%"
 			(at 167.64 95.25 90)
 			(effects
@@
 			)
 		)
-		(property "LCSC" "C346768"
+		(property "LCSC" "C912570"
 			(at 170.18 97.79 90)
 			(effects
@@
 			)
 		)
-		(property "Value" "0.22R 1%"
+		(property "Value" "0.68R 1%"
 			(at 198.12 95.25 90)
 			(effects
@@
 			)
 		)
-		(property "LCSC" "C346768"
+		(property "LCSC" "C912570"
 			(at 200.66 97.79 90)
 			(effects
