File: PCB/VORTAC/KiCAD/VORTAC_REV1/VORTAC_REV1.kicad_sch (KiCad schematic)
At the start: 0 parts

Commit message: night night
Other:
- note removed: "notes: -depletion mosfet - potenmtial candidate for reverse voltage protection (if not use p type mosfet)"
Changed lines of the file:
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@@
 		(comment 4 "-- VORTAC PCB --")
-	)
-	(text "notes:\n-depletion mosfet - potenmtial candidate for reverse voltage protection (if not use p type mosfet)"
-		(exclude_from_sim no)
-		(at 173.99 26.67 0)
-		(effects
-			(font
-				(size 1.27 1.27)
-			)
-			(justify left bottom)
-		)
 	)
 	(sheet
