File: PCB/VORTAC/KiCAD/VORTAC_REV1/VORTAC_REV1.kicad_pcb (KiCad board)
At the start: 4 copper layers, 45.6 x 32.1 mm, 79 parts, among them IC1 TMC2209-LA, J1 DEBUG, J14 918-418K2023S40001, J15 STEPPER, J2 DEBUG, J3 Conn_01x05, SW1 Boot, SW2 Reset, U1 TLV73333PDBV, U2 STM32F103C8T6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

Commit message: night night
Parts:
- removed J2: DEBUG, Connector_PinHeader_1.27mm:PinHeader_2x04_P1.27mm_Vertical
- removed JP1: Jumper, Connector_PinHeader_1.27mm:PinHeader_2x01_P1.27mm_Vertical
- added Q3: BSS138AKDW, Package_TO_SOT_SMD:SOT-363_SC-70-6, F.Cu at (158.4, 126.7)
- added R16: 10K, Resistor_SMD:R_0402_1005Metric, F.Cu at (157.7, 129.6)
- R10: value 120R -> 110R
- moved J1 29.2 mm to (116.6, 102.5), turned to -135 degrees
- moved C3 0.72 mm to (156.7, 113.1)
- renumbered HSE1 to Y1
Connections:
- J1 pad 1: BOOT_0 -> GND
- R10 pad 1: CAN_H -> CAN_L
- R10 pad 2: Net-(JP1-A) -> CAN_TRM_L
- U2 pad 42: unconnected-(U2-PB6-Pad42) -> CAN_TRM
Routing:
- added copper zone on B.Cu, net +3V3
- added copper zone on F.Cu, net GND

Commit message: BOMBOM
Parts:
- J1: footprint Vortac:PinHeader_2x03_P1.27mm_Vertical -> Connector_PinSocket_2.54mm:PinSocket_2x03_P2.54mm_Vertical
- J3: footprint Connector_PinHeader_2.54mm:PinHeader_2x03_P2.54mm_Vertical -> Connector_PinHeader_2.54mm:PinHeader_2x02_P2.54mm_Vertical
- moved J1 8.40 mm to (122.6, 108.5), turned to -45 degrees
- moved LED1 0.60 mm to (96.6, 123.2)
- moved LED2 0.60 mm to (103.4, 123.2)
Connections:
- J3 pad 2: TOOL_ID -> VDC
- J3 pad 3: VDC -> CAN_L
- J3 pad 4: CAN_L -> CAN_H
Routing:
- removed copper zone on B.Cu, net +3V3
- removed copper zone on F.Cu, net GND
Other:
- board size 45.6 x 32.1 mm -> 41.6 x 32.1 mm
