File: PCB/VORTAC/KiCAD/VORTAC_REV1/VORTAC_REV1.kicad_pcb (KiCad board)
At the start: 4 copper layers, 41.6 x 32.1 mm, 79 parts, among them IC1 TMC2209-LA, J1 DEBUG, J14 918-418K2023S40001, J15 STEPPER, J3 Conn_01x05, Q3 BSS138AKDW, SW1 Boot, SW2 Reset, U1 TLV73333PDBV, U2 STM32F103C8T6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

Commit message: Evil Mita is v00:98
Parts:
- C10, C13, C15, C2, C21, C24, C26, C28, C29: footprint Capacitor_SMD:C_0603_1608Metric -> Capacitor_SMD:C_0402_1005Metric
- C17, C19, C25, C33, C35, C36, C37, C38, C39: value 0.1uF 16V -> 0.1uF 50V
- C23: value 22nF X7R 10% 50V -> 22nF 50V; footprint Capacitor_SMD:C_0603_1608Metric -> Capacitor_SMD:C_0402_1005Metric
- C27: footprint Capacitor_SMD:C_1206_3216Metric -> Capacitor_SMD:C_0805_2012Metric
- C3, C8: value 1uF -> 1uF 16V
- C30, C31: value 22uF -> 22uF 16V
- C40: value 4.7uF 10V -> 4.7uF 50V; footprint Capacitor_SMD:C_0402_1005Metric -> Capacitor_SMD:C_0603_1608Metric
- C42, C43: value 16pF -> 16pF 50V
- J3: value Conn_01x05 -> Conn_02x02_Odd_Even
- R10: value 110R -> 115R
- R3, R4: value 5.12K -> 5.1K
- R30, R34: footprint Resistor_SMD:R_1206_3216Metric -> Resistor_SMD:R_0805_2012Metric
- R5, R6: footprint Resistor_SMD:R_0603_1608Metric -> Resistor_SMD:R_0402_1005Metric
- R7: value 100R -> 115R
- moved C34 16.1 mm to (112.7, 102.3)
- moved H1 8.94 mm to (127.5, 121.4)
- moved R14 8.11 mm to (109.0, 95.1), turned to 90 degrees
- moved C15 5.81 mm to (111.7, 95.1), turned to 90 degrees
- moved R36 5.49 mm to (116.3, 116.1)
- moved R35 5.49 mm to (116.3, 117.2)
- moved J14 3.57 mm to (120.0, 121.6)
- moved J3 0.06 mm to (118.8, 101.2)
Connections:
- J3 pad 1: GND -> VDC
- J3 pad 2: VDC -> CAN_H
- J3 pad 4: CAN_H -> GND

Commit message: No Body knows.... The trouble I've seen
Parts:
- D5, LED1, LED2, R13, R7: moved to B.Cu
- moved C30 49.4 mm to (110.2, 98.6), turned to 180 degrees
- moved C31 49.3 mm to (110.2, 100.7), turned to 180 degrees
- moved C3 48.5 mm to (109.2, 103.2), turned to -90 degrees
- moved C28 48.1 mm to (111.0, 97.1), turned to 180 degrees
- moved R5 47.8 mm to (125.2, 109.6)
- moved R8 44.0 mm to (125.2, 114.4), turned to 180 degrees
- moved C27 43.3 mm to (116.5, 98.8), turned to 90 degrees
- moved C8 42.5 mm to (115.0, 103.2), turned to -90 degrees
- moved L1 42.1 mm to (118.0, 105.2), turned to 180 degrees
- moved C25 41.8 mm to (125.2, 113.4), turned to 180 degrees
- moved U1 41.4 mm to (112.1, 103.5)
- moved U6 39.9 mm to (113.7, 98.7), turned to 90 degrees
- moved L3 39.8 mm to (113.6, 94.0), turned to 90 degrees
- moved R15 39.1 mm to (125.2, 115.5)
- moved U8 38.7 mm to (117.5, 109.0), turned to 90 degrees
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Connections:
- J3 pad 1: VDC -> GND
- J3 pad 2: CAN_H -> CAN_L
- J3 pad 3: CAN_L -> VDC
- J3 pad 4: GND -> CAN_H
- L1 pad 1: Net-(U8-CANH) -> Net-(U8-CANL)
- L1 pad 2: CAN_H -> CAN_L
- L1 pad 3: CAN_L -> CAN_H
- L1 pad 4: Net-(U8-CANL) -> Net-(U8-CANH)
- Q3 pad 3: CAN_TRM_L -> CAN_L
- Q3 pad 6: CAN_H -> CAN_TRM_H
- R10 pad 1: CAN_L -> CAN_H
- R10 pad 2: CAN_TRM_L -> CAN_TRM_H
Other:
- board size 41.6 x 32.1 mm -> 39.2 x 33.4 mm

Commit message: Nobody knows, my Sorrow...
Parts:
- C10, C13, C2, C21, C22, C23, C24, C26, C29, C33, C36, C37, C38, C39, C42, C43, D6, L1, R11, R12, R32, R38, U8: moved to B.Cu
- moved Q3 42.3 mm to (127.2, 98.2)
- moved R16 42.0 mm to (129.3, 98.6), turned to 90 degrees
- moved R10 40.5 mm to (124.0, 98.0), turned to -90 degrees
- moved C22 33.4 mm to (107.1, 108.2), turned to 90 degrees
- moved C9 32.8 mm to (100.4, 109.4), turned to 0 degrees
- moved C29 28.6 mm to (100.7, 109.7), turned to 90 degrees
- moved C42 27.4 mm to (117.2, 118.0), turned to 90 degrees
- moved C37 27.3 mm to (119.1, 112.6), turned to -90 degrees
- moved C6 27.1 mm to (100.4, 111.2)
- moved C10 26.1 mm to (100.7, 114.2), turned to -90 degrees
- moved R32 26.0 mm to (104.3, 108.2)
- moved C33 25.2 mm to (111.9, 116.5), turned to 90 degrees
- moved C39 24.9 mm to (117.6, 114.6), turned to 180 degrees
- moved C24 24.2 mm to (105.8, 108.8), turned to 90 degrees
- moved C36 23.2 mm to (115.8, 104.7)
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Routing:
- net GND: track 0.00 -> 14.1 mm, vias 0 -> 2
- net VDC: track 0.00 -> 13.3 mm
- net AS_NSS: track 0.00 -> 13.1 mm
- net AS_SCK: track 0.00 -> 12.8 mm
- net AS_MISO: track 0.00 -> 12.5 mm
- net AS_MOSI: track 0.00 -> 12.2 mm
- net +5V: track 0.00 -> 11.1 mm, vias 0 -> 2
- net STEP_1_A2: track 0.00 -> 10.4 mm
- net STEP_1_B2: track 0.00 -> 10.2 mm
- net STEP_1_A1: track 0.00 -> 8.27 mm
- net STEP_1_B1: track 0.00 -> 8.06 mm
- net Net-(LED1-DOUT): track 0.00 -> 6.62 mm
- net CAN_RX: track 0.00 -> 6.31 mm
- net CAN_TX: track 0.00 -> 5.94 mm
- net HSE_OSC_IN: track 0.00 -> 5.90 mm
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
Commit message: Girl Math
Parts:
- C15, C17, C35, C40, Q3, R10, R14, R16, R9: moved to B.Cu
- C30, C31: footprint Capacitor_SMD:C_0805_2012Metric -> Capacitor_SMD:C_0603_1608Metric
- R11: moved to F.Cu
- moved C35 26.9 mm to (114.2, 98.3)
- moved R16 18.8 mm to (111.5, 92.8)
- moved C17 18.3 mm to (119.2, 104.4), turned to 0 degrees
- moved R14 16.5 mm to (111.0, 104.8)
- moved C15 16.2 mm to (110.1, 104.8)
- moved R9 14.9 mm to (128.3, 106.6), turned to 180 degrees
- moved Q3 14.6 mm to (113.4, 93.4), turned to -90 degrees
- moved R11 14.5 mm to (116.5, 110.5)
- moved C40 12.8 mm to (119.5, 116.3), turned to 90 degrees
- moved D5 12.2 mm to (119.1, 122.4)
- moved R10 9.55 mm to (115.3, 94.1), turned to 90 degrees
- moved R8 9.44 mm to (115.9, 113.0), turned to 90 degrees
- moved R12 6.50 mm to (107.9, 110.7), turned to -90 degrees
- moved SW1 6.32 mm to (130.1, 116.1), turned to 90 degrees
- moved R3 5.73 mm to (126.7, 120.9), turned to 180 degrees
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Connections:
- J1 pad 3: NRST -> DEBUG_SWDIO
- J1 pad 4: DEBUG_SWO -> NRST
- J1 pad 5: DEBUG_SWDIO -> DEBUG_SWCLK
- J1 pad 6: DEBUG_SWCLK -> DEBUG_SWO
- J3 pad 2: CAN_L -> VDC
- J3 pad 3: VDC -> CAN_H
- J3 pad 4: CAN_H -> CAN_L
- Q3 pad 3: CAN_L -> CAN_TRM_H
- Q3 pad 6: CAN_TRM_H -> CAN_L
Routing:
- net VDC: track 13.3 -> 41.6 mm, vias 0 -> 2
- net CAN_TRM: track 0.00 -> 26.5 mm
- net USB_D+: track 0.00 -> 22.6 mm, vias 0 -> 2
- net USB_D-: track 0.00 -> 18.9 mm, vias 0 -> 1
- net Net-(D5-A): track 0.00 -> 15.2 mm
- net TMC_DIR: track 0.00 -> 10.3 mm
- net DEBUG_SWDIO: track 0.00 -> 9.62 mm, vias 0 -> 1
- net ENDSTOP_Z: track 0.00 -> 8.72 mm, vias 0 -> 1
- net TMC_STEP: track 0.00 -> 7.90 mm
- net Net-(U2-PA4): track 0.00 -> 7.58 mm, vias 0 -> 2
- net DEBUG_SWO: track 0.00 -> 7.57 mm, vias 0 -> 1
- net CAN_TX: track 5.94 -> 12.7 mm
- net CAN_H: track 0.00 -> 6.39 mm
- net CAN_RX: track 6.31 -> 12.5 mm
- net +5V: track 11.1 -> 17.3 mm, vias 2 -> 5
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- added copper zone on In1.Cu, net +3V3
- added copper zone on In1.Cu, net +5V
- added copper zone on B.Cu, net GND
- added copper zone on F.Cu, net GND
- added copper zone on In2.Cu, net GND

Commit message: Route me like one of you French girls
Parts:
- removed Q3: BSS138AKDW, Package_TO_SOT_SMD:SOT-363_SC-70-6
- removed R16: 10K, Resistor_SMD:R_0402_1005Metric
- added REF**: VORTAC_Logo_Gold, Vortac:VORTAC_Logo_Gold, F.Cu at (121.0, 115.5)
- H1, H2: footprint MountingHole:MountingHole_2.2mm_M2_Pad_Via -> Vortac:MountingHole_2.2mm_M2_Pad_Via_netless
- moved R5 6.17 mm to (128.9, 106.9)
- moved R35 5.03 mm to (114.0, 115.5)
- moved R36 5.03 mm to (115.1, 115.5)
- moved R15 3.84 mm to (123.8, 111.9), turned to -90 degrees
- moved R9 3.12 mm to (130.8, 104.7)
- moved R11 1.80 mm to (114.8, 109.7)
- moved R10 1.70 mm to (114.9, 95.8), turned to 180 degrees
- moved R8 1.60 mm to (114.8, 111.8)
- moved C13 1.52 mm to (132.6, 105.3), turned to -90 degrees
- moved C35 1.08 mm to (114.2, 99.4)
- moved R14 1.08 mm to (110.0, 104.8)
- moved C15 0.83 mm to (110.9, 104.8)
- moved C38 0.64 mm to (109.4, 107.0), turned to -90 degrees
- moved C22 0.59 mm to (107.7, 108.2)
- moved SW1 0.45 mm to (129.6, 116.1)
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Connections:
- R10 pad 2: CAN_TRM_H -> CAN_L
- U2 pad 42: CAN_TRM -> unconnected-(U2-PB6-Pad42)
Routing:
- net CAN_TRM: track 26.5 -> 0.00 mm
- net TMC_ENN: track 2.37 -> 15.7 mm, vias 0 -> 2
- net USB_D+: track 22.6 -> 12.6 mm
- net USB_D-: track 18.9 -> 8.92 mm
- net +3V3: track 11.4 -> 17.8 mm, vias 1 -> 5
- net Net-(U2-PA11): track 3.19 -> 8.18 mm
- net Net-(U2-PA12): track 3.51 -> 8.20 mm
- net VDC: track 41.6 -> 45.3 mm, vias 2 -> 3
- net CAN_L: track 5.17 -> 8.02 mm
- net Net-(IC1-5VOUT): track 0.00 -> 2.72 mm
- net Net-(Q3-S1): track 2.44 -> 0.00 mm
- net AS_NSS: track 12.6 -> 14.9 mm
- net Net-(U8-CANL): track 0.00 -> 1.72 mm
- net CAN_TRM_H: track 1.71 -> 0.00 mm
- net Net-(U8-CANH): track 0.00 -> 1.62 mm
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
Commit message: FML
Parts:
- removed REF**: VORTAC_Logo_Gold, Vortac:VORTAC_Logo_Gold
- H1, H2: footprint Vortac:MountingHole_2.2mm_M2_Pad_Via_netless -> Vortac:MountingHole_2.2mm_M2_Pad_Via_NTR
- moved C27 7.50 mm to (113.4, 92.2), turned to 180 degrees
- moved C3 7.31 mm to (114.4, 98.2), turned to 0 degrees
- moved L3 6.17 mm to (110.5, 100.0), turned to -90 degrees
- moved C30 5.81 mm to (108.8, 104.1), turned to -90 degrees
- moved U6 4.56 mm to (113.4, 94.9), turned to 180 degrees
- moved C8 3.96 mm to (111.8, 104.1), turned to -90 degrees
- moved U1 3.62 mm to (114.7, 101.0), turned to -90 degrees
- moved C31 3.59 mm to (110.3, 104.1), turned to -90 degrees
- moved C28 1.69 mm to (110.8, 96.5), turned to 90 degrees
- moved R11 0.91 mm to (115.7, 109.8)
- moved R8 0.91 mm to (115.7, 111.7)
- moved R10 0.49 mm to (114.6, 96.2)
- moved C35 0.44 mm to (114.1, 99.8)
- moved U8 0.36 mm to (116.3, 101.8)
- moved L1 0.35 mm to (115.5, 98.1)
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Connections:
- net Net-(U2-PA11) renamed /MCU/DAMPEND_USB_DL
- net Net-(U2-PA12) renamed /MCU/DAMPEND_USB_DH
- net Net-(U8-CANH) renamed /MCU/CAN_H_CHOKE
- net Net-(U8-CANL) renamed /MCU/CAN_L_CHOKE
Routing:
- net /MCU/DAMPEND_USB_DL: track 8.18 -> 3.23 mm, vias 1 -> 0
- net VDC: track 45.3 -> 41.4 mm
- net +5V: track 16.8 -> 14.6 mm
- net Net-(U6-SW): track 2.24 -> 4.35 mm
- net Net-(U6-BST): track 3.42 -> 1.53 mm
- net GND: track 13.6 -> 15.5 mm, vias 13 -> 19
- net USB_D-: track 8.92 -> 10.6 mm
- net USB_D+: track 12.6 -> 14.1 mm

Commit message: USB C Pain
Parts:
- added X1: Logo Gold, Vortac:VORTAC_Logo_Gold, F.Cu at (121.2, 114.8)
- R14, R9: moved to F.Cu
- moved R9 16.9 mm to (115.0, 110.8)
- moved R5 12.5 mm to (129.1, 119.4), turned to 180 degrees
- moved R14 8.03 mm to (109.4, 96.8), turned to 0 degrees
- moved R15 6.31 mm to (127.7, 106.9), turned to 0 degrees
- moved C25 4.85 mm to (125.8, 108.6), turned to 90 degrees
- moved R11 2.14 mm to (115.0, 111.8), turned to 180 degrees
- moved R8 1.96 mm to (115.0, 109.9), turned to 0 degrees
- moved C13 1.11 mm to (131.9, 106.1)
- moved C15 0.80 mm to (110.2, 104.3), turned to 0 degrees
- moved R35 0.09 mm to (114.1, 115.5)
- moved R36 0.05 mm to (115.0, 115.5)
- turned U7 to 90 degrees
Connections:
- net /MCU/DAMPEND_USB_DH renamed /MCU/DAMPEND_USB_D+
- net /MCU/DAMPEND_USB_DL renamed /MCU/DAMPEND_USB_D-
Routing:
- net /MCU/DAMPEND_USB_D-: track 3.23 -> 8.21 mm, vias 0 -> 1
- net USB_D-: track 10.6 -> 15.0 mm
- net USB_D+: track 14.1 -> 17.0 mm, vias 2 -> 3
- net GND: track 15.5 -> 16.8 mm, vias 19 -> 20
- net Net-(D5-A): track 14.4 -> 15.4 mm
- net +5V: track 14.6 -> 13.7 mm, vias 5 -> 4
- net +3V3: track 17.5 -> 16.6 mm
- net AS_NSS: track 14.8 -> 14.5 mm, vias 0 -> 1
Other:
- board text added: "Use Stackup JLC041011-7628(Standard/Finished thickness0.99±0.10mm) For 0.2mm prepreg dialectic between outer layers"

Commit message: USB C Survivor
Parts:
- moved SW1 6.25 mm to (126.7, 110.6), turned to -45 degrees
- moved R36 5.70 mm to (115.0, 109.8), turned to 0 degrees
- moved R35 4.84 mm to (115.0, 110.7), turned to 0 degrees
- moved SW2 3.06 mm to (128.9, 108.3), turned to -45 degrees
- moved R9 2.72 mm to (115.0, 113.5), turned to 0 degrees
- moved R8 1.77 mm to (115.0, 111.7)
- moved R11 0.82 mm to (115.0, 112.6)
- moved C17 0.52 mm to (119.2, 103.6)
- moved X1 0.50 mm to (121.4, 115.3)
- moved R4 0.50 mm to (122.4, 122.5)
- moved R3 0.48 mm to (127.1, 120.8)
- turned C13 to -45 degrees
Routing:
- net NRST: track 1.04 -> 19.1 mm
- net USB_D-: track 15.0 -> 28.4 mm, vias 1 -> 2
- net ENDSTOP_X: track 3.41 -> 13.9 mm
- net USB_D+: track 17.0 -> 25.2 mm, vias 3 -> 1
- net /MCU/DAMPEND_USB_D+: track 8.20 -> 4.07 mm
- net /MCU/DAMPEND_USB_D-: track 8.21 -> 5.16 mm
- net GND: track 16.8 -> 14.2 mm
- net Net-(U7-ANODE): track 0.00 -> 2.48 mm
- net Net-(U7-OUTPUT): track 0.00 -> 1.85 mm
- net Net-(D5-A): track 15.4 -> 14.4 mm
- net Net-(J14-CC1): track 2.29 -> 2.90 mm
- net Net-(J14-CC2): track 2.40 -> 1.80 mm
