File: PCB/VORTAC/KiCAD/VORTAC_REV1/Headers.kicad_sch (KiCad schematic)
At the start: 10 parts, among them J1 DEBUG, J14 918-418K2023S40001, J15 STEPPER, J2 DEBUG, J3 Conn_01x05

Commit message: Schematic Updates - Changed the 5V Rail to a more space efficient implementation
Parts:
- J15: footprint Vortac:JST_PH_S4B-PH-K_1x04_P2.00mm_Horizontal -> Vortac:Motor_Hand_Wire_pads; LCSC C144395 -> (none)
- J2: footprint (none) -> Connector_PinHeader_1.27mm:PinHeader_2x04_P1.27mm_Vertical
Changed lines of the file:
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@@
 			)
 		)
-		(property "Footprint" "Vortac:JST_PH_S4B-PH-K_1x04_P2.00mm_Horizontal"
+		(property "Footprint" "Vortac:Motor_Hand_Wire_pads"
 			(at 48.26 29.21 0)
 			(effects
@@
 			)
 		)
-		(property "LCSC" "C144395"
+		(property "LCSC" ""
 			(at 48.26 29.21 0)
 			(effects
@@
 			)
 		)
-		(property "Footprint" ""
+		(property "Footprint" "Connector_PinHeader_1.27mm:PinHeader_2x04_P1.27mm_Vertical"
 			(at 46.99 71.12 0)
 			(effects

Commit message: update to Kicad 9.0.X
Changed lines of the file:
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@@
 (kicad_sch
-	(version 20231120)
+	(version 20250114)
 	(generator "eeschema")
-	(generator_version "8.0")
+	(generator_version "9.0")
 	(paper "A4")
 	(title_block
@@
 		(comment 4 "-- VORTAC PCB --")
 	)
+	(rectangle
+		(start 16.51 44.45)
+		(end 83.82 80.01)
+		(stroke
+			(width 0)
+			(type dash)
+		)
+		(fill
+			(type none)
+		)
+	)
+	(text "todo:\n- consider connector selection\n- consider combining fan or io/led headers\n- remove duplicate heater/thermistor header\n- add probepoints\n- change usb-c symbol (sucks bro)"
+		(exclude_from_sim no)
+		(at 233.68 179.07 0)
+		(effects
+			(font
+				(size 1.27 1.27)
+			)
+			(justify left bottom)
+		)
+	)
+	(text "Connection to Daughterboard"
+		(exclude_from_sim no)
+		(at 27.686 119.38 0)
+		(effects
+			(font
+				(size 1.27 1.27)
+			)
+			(justify left bottom)
+		)
+	)
+	(text "Tool Interface"
+		(exclude_from_sim no)
+		(at 27.432 89.154 0)
+		(effects
+			(font
+				(size 1.8034 1.8034)
+			)
+			(justify left bottom)
+		)
+	)
+	(text "Stepper Header"
+		(exclude_from_sim no)
+		(at 20.32 21.59 0)
+		(effects
+			(font
+				(size 1.8034 1.8034)
+			)
+			(justify left bottom)
+		)
+	)
+	(text "BOOT_1 optional for SRAM boot\nIf not included a sjumper it could be \naccessed by soldering to the resistor when needed"
+		(exclude_from_sim no)
+		(at 103.632 52.832 0)
+		(effects
+			(font
+				(size 0.7874 0.7874)
+			)
+			(justify left top)
+		)
+	)
+	(text "Debug Header"
+		(exclude_from_sim no)
+		(at 20.574 50.546 0)
+		(effects
+			(font
+				(size 1.8034 1.8034)
+			)
+			(justify left bottom)
+		)
+	)
+	(text "Type C USB 2.0"
+		(exclude_from_sim no)
+		(at 20.32 130.81 0)
+		(effects
+			(font
+				(size 1.8034 1.8034)
+			)
+			(justify left bottom)
+		)
+	)
+	(text "ESD Protection for Shield could be added\n(other design add a cap and resistor to ground)"
+		(exclude_from_sim no)
+		(at 20.32 188.468 0)
+		(effects
+			(font
+				(size 1.27 1.27)
+			)
+			(justify left bottom)
+		)
+	)
 	(junction
 		(at 31.75 179.07)
@@
 		)
 	)
-	(rectangle
-		(start 16.51 44.45)
-		(end 83.82 80.01)
-		(stroke
-			(width 0)
-			(type dash)
-		)
-		(fill
-			(type none)
-		)
-	)
-	(text "todo:\n- consider connector selection\n- consider combining fan or io/led headers\n- remove duplicate heater/thermistor header\n- add probepoints\n- change usb-c symbol (sucks bro)"
-		(exclude_from_sim no)
-		(at 233.68 179.07 0)
-		(effects
-			(font
-				(size 1.27 1.27)
-			)
-			(justify left bottom)
-		)
-	)
-	(text "Connection to Daughterboard"
-		(exclude_from_sim no)
-		(at 27.686 119.38 0)
-		(effects
-			(font
-				(size 1.27 1.27)
-			)
-			(justify left bottom)
-		)
-	)
-	(text "Tool Interface"
-		(exclude_from_sim no)
-		(at 27.432 89.154 0)
-		(effects
-			(font
-				(size 1.8034 1.8034)
-			)
-			(justify left bottom)
-		)
-	)
-	(text "Stepper Header"
-		(exclude_from_sim no)
-		(at 20.32 21.59 0)
-		(effects
-			(font
-				(size 1.8034 1.8034)
-			)
-			(justify left bottom)
-		)
-	)
-	(text "BOOT_1 optional for SRAM boot\nIf not included a sjumper it could be \naccessed by soldering to the resistor when needed"
-		(exclude_from_sim no)
-		(at 103.632 52.832 0)
-		(effects
-			(font
-				(size 0.7874 0.7874)
-			)
-			(justify left top)
-		)
-	)
-	(text "Debug Header"
-		(exclude_from_sim no)
-		(at 20.574 50.546 0)
-		(effects
-			(font
-				(size 1.8034 1.8034)
-			)
-			(justify left bottom)
-		)
-	)
-	(text "Type C USB 2.0"
-		(exclude_from_sim no)
-		(at 20.32 130.81 0)
-		(effects
-			(font
-				(size 1.8034 1.8034)
-			)
-			(justify left bottom)
-		)
-	)
-	(text "ESD Protection for Shield could be added\n(other design add a cap and resistor to ground)"
-		(exclude_from_sim no)
-		(at 20.32 188.468 0)
-		(effects
-			(font
-				(size 1.27 1.27)
-			)
-			(justify left bottom)
-		)
-	)

Commit message: Update Symbol Librarys
Parts:
- J14: symbol VORTAC-rescue:USB_C_Receptacle_USB2.0-Connector -> Vortac:USB_C_Receptacle_USB2.0-Connector
Changed lines of the file:
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@@
 	)
 	(symbol
-		(lib_id "VORTAC-rescue:USB_C_Receptacle_USB2.0-Connector")
+		(lib_id "Vortac:USB_C_Receptacle_USB2.0-Connector")
 		(at 31.75 156.21 0)
 		(unit 1)
@@
 		(dnp no)
 		(property "Reference" "J14"
-			(at 34.4678 134.1882 0)
-			(effects
-				(font
-					(size 1.27 1.27)
-				)
+			(at 21.59 137.16 0)
+			(effects
+				(font
+					(size 1.27 1.27)
+				)
+				(justify left)
 			)
 		)
@@
 	)
 	(symbol
-		(lib_id "VORTAC-rescue:GND-power")
+		(lib_id "power:GND")
 		(at 63.5 179.07 90)
 		(unit 1)
@@
 		(on_board yes)
 		(dnp no)
-		(property "Reference" "#PWR09"
+		(property "Reference" "#PWR9"
 			(at 69.85 179.07 0)
 			(effects
@@
 			)
 		)
-		(property "Description" ""
+		(property "Description" "Power symbol creates a global label with name \"GND\" , ground"
 			(at 63.5 179.07 0)
 			(effects
@@
 			(project "VORTAC_REV1"
 				(path "/ed58d858-d9f9-4504-a982-ccfc7f9efbad/00000000-0000-0000-0000-0000613db78d"
-					(reference "#PWR09")
+					(reference "#PWR9")
 					(unit 1)
 				)
@@
 	)
 	(symbol
-		(lib_id "VORTAC-rescue:GND-power")
+		(lib_id "power:GND")
 		(at 39.37 109.22 90)
 		(unit 1)
@@
 		(on_board yes)
 		(dnp no)
-		(property "Reference" "#PWR0120"
+		(property "Reference" "#PWR120"
 			(at 45.72 109.22 0)
 			(effects
@@
 			)
 		)
-		(property "Description" ""
+		(property "Description" "Power symbol creates a global label with name \"GND\" , ground"
 			(at 39.37 109.22 0)
 			(effects
@@
 			(project "VORTAC_REV1"
 				(path "/ed58d858-d9f9-4504-a982-ccfc7f9efbad/00000000-0000-0000-0000-0000613db78d"
-					(reference "#PWR0120")
-					(unit 1)
-				)
-			)
-		)
-	)
-	(symbol
-		(lib_id "VORTAC-rescue:+5V-power")
+					(reference "#PWR120")
+					(unit 1)
+				)
+			)
+		)
+	)
+	(symbol
+		(lib_id "power:+5V")
 		(at 63.5 140.97 270)
 		(unit 1)
@@
 		(on_board yes)
 		(dnp no)
-		(property "Reference" "#PWR0138"
+		(property "Reference" "#PWR138"
 			(at 59.69 140.97 0)
 			(effects
@@
 			)
 		)
-		(property "Description" ""
+		(property "Description" "Power symbol creates a global label with name \"+5V\""
 			(at 63.5 140.97 0)
 			(effects
@@
 			(project "VORTAC_REV1"
 				(path "/ed58d858-d9f9-4504-a982-ccfc7f9efbad/00000000-0000-0000-0000-0000613db78d"
-					(reference "#PWR0138")
-					(unit 1)
-				)
-			)
-		)
-	)
-	(symbol
-		(lib_id "VORTAC-rescue:+3.3V-power")
+					(reference "#PWR138")
+					(unit 1)
+				)
+			)
+		)
+	)
+	(symbol
+		(lib_id "power:+3V3")
 		(at 57.15 54.61 270)
 		(unit 1)
@@
 		(on_board yes)
 		(dnp no)
-		(property "Reference" "#PWR0160"
+		(property "Reference" "#PWR160"
 			(at 53.34 54.61 0)
 			(effects
@@
 			)
 		)
-		(property "Description" ""
+		(property "Description" "Power symbol creates a global label with name \"+3V3\""
 			(at 57.15 54.61 0)
 			(effects
@@
 			(project "VORTAC_REV1"
 				(path "/ed58d858-d9f9-4504-a982-ccfc7f9efbad/00000000-0000-0000-0000-0000613db78d"
-					(reference "#PWR0160")
-					(unit 1)
-				)
-			)
-		)
-	)
-	(symbol
-		(lib_id "VORTAC-rescue:GND-power")
+					(reference "#PWR160")
+					(unit 1)
+				)
+			)
+		)
+	)
+	(symbol
+		(lib_id "power:GND")
 		(at 138.43 33.02 0)
 		(unit 1)
@@
 		(on_board yes)
 		(dnp no)
-		(property "Reference" "#PWR029"
+		(property "Reference" "#PWR29"
 			(at 138.43 39.37 0)
 			(effects
@@
 			)
 		)
-		(property "Description" ""
+		(property "Description" "Power symbol creates a global label with name \"GND\" , ground"
 			(at 138.43 33.02 0)
 			(effects
@@
 			(project "VORTAC_REV1"
 				(path "/ed58d858-d9f9-4504-a982-ccfc7f9efbad/00000000-0000-0000-0000-0000613db78d"
-					(reference "#PWR029")
-					(unit 1)
-				)
-			)
-		)
-	)
-	(symbol
-		(lib_name "MountingHole_Pad_1")
+					(reference "#PWR29")
+					(unit 1)
+				)
+			)
+		)
+	)
+	(symbol
 		(lib_id "Mechanical:MountingHole_Pad")
 		(at 113.03 26.67 0)
@@
 		(dnp no)
 		(fields_autoplaced yes)
-		(property "Reference" "#PWR01"
+		(property "Reference" "#PWR1"
 			(at 35.56 104.14 0)
 			(effects
@@
 			(project "VORTAC_REV1"
 				(path "/ed58d858-d9f9-4504-a982-ccfc7f9efbad/00000000-0000-0000-0000-0000613db78d"
-					(reference "#PWR01")
-					(unit 1)
-				)
-			)
-		)
-	)
-	(symbol
-		(lib_id "VORTAC-rescue:GND-power")
+					(reference "#PWR1")
+					(unit 1)
+				)
+			)
+		)
+	)
+	(symbol
+		(lib_id "power:GND")
 		(at 113.03 33.02 0)
 		(unit 1)
@@
 		(on_board yes)
 		(dnp no)
-		(property "Reference" "#PWR027"
+		(property "Reference" "#PWR27"
 			(at 113.03 39.37 0)
 			(effects
@@
 			)
 		)
-		(property "Description" ""
+		(property "Description" "Power symbol creates a global label with name \"GND\" , ground"
 			(at 113.03 33.02 0)
 			(effects
@@
 			(project "VORTAC_REV1"
 				(path "/ed58d858-d9f9-4504-a982-ccfc7f9efbad/00000000-0000-0000-0000-0000613db78d"
-					(reference "#PWR027")
-					(unit 1)
-				)
+					(reference "#PWR27")
+					(unit 1)
+				)

Commit message: updated revs fabrication test
Other:
- moved on the sheet: H1, H2, J2
Changed lines of the file:
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@@
 	(wire
 		(pts
-			(xy 113.03 29.21) (xy 113.03 33.02)
+			(xy 77.47 30.48) (xy 77.47 34.29)
 		)
 		(stroke
@@
 	(wire
 		(pts
-			(xy 138.43 29.21) (xy 138.43 33.02)
+			(xy 102.87 30.48) (xy 102.87 34.29)
 		)
 		(stroke
@@
 		(dnp no)
 		(property "Reference" "J1"
-			(at 45.212 51.054 0)
+			(at 44.45 51.054 0)
 			(effects
 				(font
@@
 		)
 		(property "Value" "DEBUG"
-			(at 50.292 51.054 0)
+			(at 49.784 51.054 0)
 			(effects
 				(font
@@
 	(symbol
 		(lib_id "power:GND")
-		(at 138.43 33.02 0)
+		(at 102.87 34.29 0)
 		(unit 1)
 		(exclude_from_sim no)
@@
 		(dnp no)
 		(property "Reference" "#PWR29"
-			(at 138.43 39.37 0)
+			(at 102.87 40.64 0)
 			(effects
 				(font
@@
 		)
 		(property "Value" "GND"
-			(at 145.034 33.782 0)
+			(at 109.474 35.052 0)
 			(effects
 				(font
@@
 		)
 		(property "Footprint" ""
-			(at 138.43 33.02 0)
+			(at 102.87 34.29 0)
 			(effects
 				(font
@@
 		)
 		(property "Datasheet" ""
-			(at 138.43 33.02 0)
+			(at 102.87 34.29 0)
 			(effects
 				(font
@@
 		)
 		(property "Description" "Power symbol creates a global label with name \"GND\" , ground"
-			(at 138.43 33.02 0)
+			(at 102.87 34.29 0)
 			(effects
 				(font
@@
 	(symbol
 		(lib_id "Mechanical:MountingHole_Pad")
-		(at 113.03 26.67 0)
+		(at 77.47 27.94 0)
 		(unit 1)
 		(exclude_from_sim no)
@@
 		(fields_autoplaced yes)
 		(property "Reference" "H1"
-			(at 115.57 24.1299 0)
+			(at 80.01 25.3999 0)
 			(effects
 				(font
@@
 		)
 		(property "Value" "MountingHole_Pad"
-			(at 115.57 26.6699 0)
+			(at 80.01 27.9399 0)
 			(effects
 				(font
@@
 		)
 		(property "Footprint" "MountingHole:MountingHole_2.2mm_M2_Pad_Via"
-			(at 113.03 26.67 0)
+			(at 77.47 27.94 0)
 			(effects
 				(font
@@
 		)
 		(property "Datasheet" "~"
-			(at 113.03 26.67 0)
+			(at 77.47 27.94 0)
 			(effects
 				(font
@@
 		)
 		(property "Description" "Mounting Hole with connection"
-			(at 113.03 26.67 0)
+			(at 77.47 27.94 0)
 			(effects
 				(font
@@
 	(symbol
 		(lib_id "Connector_Generic:Conn_02x04_Odd_Even")
-		(at 46.99 71.12 0)
+		(at 46.99 68.58 0)
 		(unit 1)
 		(exclude_from_sim no)
@@
 		(dnp no)
 		(property "Reference" "J2"
-			(at 46.228 64.516 0)
+			(at 46.99 63.5 0)
 			(effects
 				(font
@@
 		)
 		(property "Value" "DEBUG"
-			(at 51.816 64.516 0)
+			(at 48.514 76.454 0)
 			(effects
 				(font
@@
 		)
 		(property "Footprint" "Connector_PinHeader_1.27mm:PinHeader_2x04_P1.27mm_Vertical"
-			(at 46.99 71.12 0)
+			(at 46.99 68.58 0)
 			(effects
 				(font
@@
 		)
 		(property "Datasheet" "~"
-			(at 46.99 71.12 0)
+			(at 46.99 68.58 0)
 			(effects
 				(font
@@
 		)
 		(property "Description" "Generic connector, double row, 02x04, odd/even pin numbering scheme (row 1 odd numbers, row 2 even numbers), script generated (kicad-library-utils/schlib/autogen/connector/)"
-			(at 46.99 71.12 0)
+			(at 46.99 68.58 0)
 			(effects
 				(font
@@
 	(symbol
 		(lib_id "power:GND")
-		(at 113.03 33.02 0)
+		(at 77.47 34.29 0)
 		(unit 1)
 		(exclude_from_sim no)
@@
 		(dnp no)
 		(property "Reference" "#PWR27"
-			(at 113.03 39.37 0)
+			(at 77.47 40.64 0)
 			(effects
 				(font
@@
 		)
 		(property "Value" "GND"
-			(at 119.634 33.782 0)
+			(at 84.074 35.052 0)
 			(effects
 				(font
@@
 		)
 		(property "Footprint" ""
-			(at 113.03 33.02 0)
+			(at 77.47 34.29 0)
 			(effects
 				(font
@@
 		)
 		(property "Datasheet" ""
-			(at 113.03 33.02 0)
+			(at 77.47 34.29 0)
 			(effects
 				(font
@@
 		)
 		(property "Description" "Power symbol creates a global label with name \"GND\" , ground"
-			(at 113.03 33.02 0)
+			(at 77.47 34.29 0)
 			(effects
 				(font
@@
 	(symbol
 		(lib_id "Mechanical:MountingHole_Pad")
-		(at 138.43 26.67 0)
+		(at 102.87 27.94 0)
 		(unit 1)
 		(exclude_from_sim no)
@@
 		(fields_autoplaced yes)
 		(property "Reference" "H2"
-			(at 140.97 24.1299 0)
+			(at 105.41 25.3999 0)
 			(effects
 				(font
@@
 		)
 		(property "Value" "MountingHole_Pad"
-			(at 140.97 26.6699 0)
+			(at 105.41 27.9399 0)
 			(effects
 				(font
@@
 		)
 		(property "Footprint" "MountingHole:MountingHole_2.2mm_M2_Pad_Via"
-			(at 138.43 26.67 0)
+			(at 102.87 27.94 0)
 			(effects
 				(font
@@
 		)
 		(property "Datasheet" "~"
-			(at 138.43 26.67 0)
+			(at 102.87 27.94 0)
 			(effects
 				(font
@@
 		)
 		(property "Description" "Mounting Hole with connection"
-			(at 138.43 26.67 0)
-			(effects
-				(font
+			(at 102.87 27.94 0)
+			(effects
+				(font

Commit message: night night
Parts:
- removed J2: DEBUG, Connector_PinHeader_1.27mm:PinHeader_2x04_P1.27mm_Vertical, symbol Connector_Generic:Conn_02x04_Odd_Even
Connections:
- net BOOT_0 is gone; now on net GND: J1.1 (Pin_1)
Other:
- note removed: "BOOT_1 optional for SRAM boot If not included a sjumper it could be accessed by soldering to the resistor when needed"

Commit message: BOMBOM
Parts:
- J1: footprint Vortac:PinHeader_2x03_P1.27mm_Vertical -> Connector_PinSocket_2.54mm:PinSocket_2x03_P2.54mm_Vertical
- J3: footprint Connector_PinHeader_2.54mm:PinHeader_2x03_P2.54mm_Vertical -> Connector_PinHeader_2.54mm:PinHeader_2x02_P2.54mm_Vertical
Connections:
- net TOOL_ID is gone; now on net VDC: J3.2 (Pin_2)
- net CAN_H: now also J3.4 (Pin_4); no longer J3.5 (Pin_5)
- net CAN_L: now also J3.3 (Pin_3); no longer J3.4 (Pin_4)
- net VDC: no longer J3.3 (Pin_3)
Other:
- moved on the sheet: J1

Commit message: Anned Parts
Parts:
- removed J3: Conn_01x05, Connector_PinHeader_2.54mm:PinHeader_2x02_P2.54mm_Vertical, symbol Connector_Generic:Conn_01x05
- added J3: Conn_02x02_Odd_Even, Connector_PinHeader_2.54mm:PinHeader_2x02_P2.54mm_Vertical, symbol Connector_Generic:Conn_02x02_Odd_Even
- D5: LCSC C37049 -> C7420331
- J1: LCSC (none) -> C2840016
- R3, R4: value 5.12K -> 5.1K; LCSC (none) -> C105872
Connections:
- net CAN_H: now also J3.2 (Pin_2)
- net CAN_L: now also J3.3 (Pin_3)
- net GND: now also J3.4 (Pin_4)
- net VDC: now also J3.1 (Pin_1)
Changed lines of the file:
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@@
-		)
-	)
-	(wire
-		(pts
-			(xy 35.56 101.6) (xy 39.37 101.6)
-		)
-		(stroke
-			(width 0)
-			(type default)
-		)
-	)
-	(wire
-		(pts
-			(xy 35.56 106.68) (xy 39.37 106.68)
-		)
-		(stroke
-			(width 0)
-			(type default)
 		)
 	)
@@
 	(wire
 		(pts
-			(xy 35.56 109.22) (xy 39.37 109.22)
+			(xy 50.8 104.14) (xy 54.61 104.14)
 		)
 		(stroke
@@
 	(wire
 		(pts
-			(xy 35.56 104.14) (xy 39.37 104.14)
-		)
-		(stroke
-			(width 0)
-			(type default)
-		)
-	)
-	(wire
-		(pts
 			(xy 52.07 179.07) (xy 52.07 168.91)
 		)
@@
 	(wire
 		(pts
+			(xy 71.12 101.6) (xy 67.31 101.6)
+		)
+		(stroke
+			(width 0)
+			(type default)
+		)
+	)
+	(wire
+		(pts
 			(xy 52.07 163.83) (xy 52.07 146.05)
 		)
@@
 	(wire
 		(pts
+			(xy 69.85 104.14) (xy 67.31 104.14)
+		)
+		(stroke
+			(width 0)
+			(type default)
+		)
+	)
+	(wire
+		(pts
 			(xy 43.18 63.5) (xy 40.64 63.5)
 		)
@@
 			(width 0)
 			(type dash)
+		)
+	)
+	(wire
+		(pts
+			(xy 50.8 101.6) (xy 54.61 101.6)
+		)
+		(stroke
+			(width 0)
+			(type default)
 		)
 	)
@@
 	(global_label "CAN_L"
 		(shape input)
-		(at 39.37 104.14 0)
+		(at 50.8 104.14 180)
 		(effects
 			(font
 				(size 1.27 1.27)
 			)
-			(justify left)
+			(justify right)
 		)
 		(property "Intersheetrefs" "${INTERSHEET_REFS}"
-			(at 39.37 104.14 0)
+			(at 50.8 104.14 0)
 			(effects
 				(font
@@
 	(global_label "CAN_H"
 		(shape input)
-		(at 39.37 101.6 0)
+		(at 71.12 101.6 0)
 		(effects
 			(font
@@
 		)
 		(property "Intersheetrefs" "${INTERSHEET_REFS}"
-			(at 39.37 101.6 0)
+			(at 71.12 101.6 0)
 			(effects
 				(font
@@
 			)
 		)
-		(property "Value" "5.12K"
+		(property "Value" "5.1K"
 			(at 54.61 173.99 90)
 			(effects
@@
 				)
 				(hide yes)
+			)
+		)
+		(property "LCSC" "C105872"
+			(at 49.53 173.99 0)
+			(effects
+				(font
+					(size 1.27 1.27)
+				)
 			)
 		)
@@
 			)
 		)
-		(property "Value" "5.12K"
+		(property "Value" "5.1K"
 			(at 55.0164 166.37 90)
 			(effects
@@
 				)
 				(hide yes)
+			)
+		)
+		(property "LCSC" "C105872"
+			(at 52.07 166.37 0)
+			(effects
+				(font
+					(size 1.27 1.27)
+				)
 			)
 		)
@@
 			)
 		)
-		(property "LCSC" "C37049"
+		(property "LCSC" "C7420331"
 			(at 55.88 140.97 0)
 			(effects
@@
 			)
 		)
+		(property "LCSC" "C2840016"
+			(at 48.26 63.5 0)
+			(effects
+				(font
+					(size 1.27 1.27)
+				)
+			)
+		)
 		(pin "3"
 		)
@@
 	(symbol
 		(lib_id "power:GND")
-		(at 39.37 109.22 90)
+		(at 69.85 104.14 90)
 		(unit 1)
 		(exclude_from_sim no)
@@
 		(dnp no)
 		(property "Reference" "#PWR120"
-			(at 45.72 109.22 0)
+			(at 76.2 104.14 0)
 			(effects
 				(font
@@
 		)
 		(property "Value" "GND"
-			(at 42.6212 109.093 90)
+			(at 73.1012 104.013 90)
 			(effects
 				(font
@@
 		)
 		(property "Footprint" ""
-			(at 39.37 109.22 0)
+			(at 69.85 104.14 0)
 			(effects
 				(font
@@
 		)
 		(property "Datasheet" ""
-			(at 39.37 109.22 0)
+			(at 69.85 104.14 0)
 			(effects
 				(font
@@
 		)
 		(property "Description" "Power symbol creates a global label with name \"GND\" , ground"
-			(at 39.37 109.22 0)
+			(at 69.85 104.14 0)
 			(effects
 				(font
@@
 	)
 	(symbol
-		(lib_id "Connector_Generic:Conn_01x05")
-		(at 30.48 104.14 180)
-		(unit 1)
-		(exclude_from_sim no)
-		(in_bom yes)
-		(on_board yes)
-		(dnp no)
-		(fields_autoplaced yes)
-		(property "Reference" "J3"
-			(at 30.48 92.71 0)
-			(effects
-				(font
-					(size 1.27 1.27)
-				)
-			)
-		)
-		(property "Value" "Conn_01x05"
-			(at 30.48 95.25 0)
-			(effects
-				(font
-					(size 1.27 1.27)
-				)
-			)
-		)
-		(property "Footprint" "Connector_PinHeader_2.54mm:PinHeader_2x02_P2.54mm_Vertical"
-			(at 30.48 104.14 0)
-			(effects
-				(font
-					(size 1.27 1.27)
-				)
-				(hide yes)
-			)
-		)
-		(property "Datasheet" "~"
-			(at 30.48 104.14 0)
-			(effects
-				(font
-					(size 1.27 1.27)
-				)
-				(hide yes)
-			)
-		)
-		(property "Description" "Generic connector, single row, 01x05, script generated (kicad-library-utils/schlib/autogen/connector/)"
-			(at 30.48 104.14 0)
-			(effects
-				(font
-					(size 1.27 1.27)
-				)
-				(hide yes)
-			)
-		)
-		(pin "5"
-		)
-		(pin "2"
-		)
-		(pin "3"
-		)
-		(pin "1"
-		)
-		(pin "4"
-		)
-		(instances
-			(project "VORTAC_REV1"
-				(path "/ed58d858-d9f9-4504-a982-ccfc7f9efbad/00000000-0000-0000-0000-0000613db78d"
-					(reference "J3")
-					(unit 1)
-				)
-			)
-		)
-	)
-	(symbol
 		(lib_id "power:GND")
 		(at 40.64 60.96 270)
@@
 	)
 	(symbol
-		(lib_id "power:VDC")
-		(at 39.37 106.68 270)
+		(lib_id "Connector_Generic:Conn_02x02_Odd_Even")
+		(at 59.69 101.6 0)
 		(unit 1)
 		(exclude_from_sim no)
@@
 		(dnp no)
 		(fields_autoplaced yes)
+		(property "Reference" "J3"
+			(at 60.96 95.25 0)
+			(effects
+				(font
+					(size 1.27 1.27)
+				)
+			)
+		)
+		(property "Value" "Conn_02x02_Odd_Even"
+			(at 60.96 97.79 0)
+			(effects
+				(font
+					(size 1.27 1.27)
+				)
+			)
+		)
+		(property "Footprint" "Connector_PinHeader_2.54mm:PinHeader_2x02_P2.54mm_Vertical"
+			(at 59.69 101.6 0)
+			(effects
+				(font
+					(size 1.27 1.27)
+				)
+				(hide yes)
+			)
+		)
+		(property "Datasheet" "~"
+			(at 59.69 101.6 0)
+			(effects
+				(font
+					(size 1.27 1.27)
+				)
+				(hide yes)
+			)
+		)
+		(property "Description" "Generic connector, double row, 02x02, odd/even pin numbering scheme (row 1 odd numbers, row 2 even numbers), script generated (kicad-library-utils/schlib/autogen/connector/)"
+			(at 59.69 101.6 0)
+			(effects
+				(font
+					(size 1.27 1.27)
+				)
+				(hide yes)
+			)
+		)
+		(property "LCSC" "C7501273"
+			(at 59.69 101.6 0)
+			(effects
+				(font
+					(size 1.27 1.27)
+				)
+			)
+		)
+		(pin "1"
+		)
+		(pin "3"
+		)
+		(pin "4"
+		)
+		(pin "2"
+		)
+		(instances
+			(project ""
+				(path "/ed58d858-d9f9-4504-a982-ccfc7f9efbad/00000000-0000-0000-0000-0000613db78d"
+					(reference "J3")
+					(unit 1)
+				)
+			)
+		)
+	)
+	(symbol
+		(lib_id "power:VDC")
+		(at 50.8 101.6 90)
+		(unit 1)
+		(exclude_from_sim no)
+		(in_bom yes)
+		(on_board yes)
+		(dnp no)
 		(property "Reference" "#PWR1"
-			(at 35.56 106.68 0)
+			(at 54.61 101.6 0)
 			(effects
 				(font
@@
 		)
 		(property "Value" "VDC"
-			(at 43.18 106.6799 90)
-			(effects
-				(font
-					(size 1.27 1.27)
-				)
-				(justify left)
+			(at 45.466 99.822 90)
+			(effects
+				(font
+					(size 1.27 1.27)
+				)
 			)
 		)
 		(property "Footprint" ""
-			(at 39.37 106.68 0)
+			(at 50.8 101.6 0)
 			(effects
 				(font
@@
 		)
 		(property "Datasheet" ""
-			(at 39.37 106.68 0)
+			(at 50.8 101.6 0)
 			(effects
 				(font
@@
 		)
 		(property "Description" "Power symbol creates a global label with name \"VDC\""
-			(at 39.37 106.68 0)
-			(effects
-				(font
+			(at 50.8 101.6 0)
+			(effects
+				(font
