File: PCB/VORTAC/KiCAD/VORTAC_REV1/Logic.kicad_sch (KiCad schematic)
At the start: 34 parts, among them U1 TLV73333PDBV, U3 EE-SX4320, U4 TPS54335ADRCR, U5 AS5047D, U7 EE-SX3350

Commit message: Schematic Updates - Changed the 5V Rail to a more space efficient implementation
Parts:
- removed D1: SK6812, LED_SMD:LED_SK6812_PLCC4_5.0x5.0mm_P3.2mm, symbol LED:SK6812
- removed R1, R7: 1K, Resistor_SMD:R_0603_1608Metric, symbol Device:R
- added C27: 10uF 50V, Capacitor_SMD:C_1206_3216Metric, symbol Device:C_Small
- added C28: 0.1uF 50V, Capacitor_SMD:C_0603_1608Metric, symbol Device:C_Small
- added C30, C31: 22uF, Capacitor_SMD:C_0805_2012Metric, symbol Device:C_Small
- added L3: 4.7uH, Vortac:L_Sunlord_MWSA0518_5.4x5.2mm, symbol Device:L
- added LED1, LED2: SK6812SIDE-A-RVS, Vortac:LED-SMD_4P-L4.0-W1.6-L, symbol Vortac:SK6812SIDE-A-RVS
- added R1, R15: 1K, Resistor_SMD:R_0402_1005Metric, symbol Device:R_Small
- added U6: AP63205WU, Package_TO_SOT_SMD:TSOT-23-6, symbol Regulator_Switching:AP63205WU
- added U9: TPS54202DDC, Package_TO_SOT_SMD:SOT-23-6, symbol Regulator_Switching:TPS54202DDC
Connections:
- net +5V: now also C30.1, C31.1, L3.2, LED1.2 (VDD), LED2.2 (VDD), U6.1 (FB)
- net ENDSTOP_X: now also R15.1
- net ENDSTOP_Z: now also R1.1
- net GND: now also C27.2, C30.2, C31.2, LED1.4 (GND), LED2.4 (GND), U6.4 (GND)
- net VDC: now also C27.1, U6.2 (EN), U6.3 (IN)
- net at U3.6 (OUTPUT): now also R1.2
- net at U7.5 (OUTPUT): now also R15.2
- new net: LED1.3 (DOUT), LED2.1 (DIN)
- new net: C28.2, L3.1, U6.5 (SW)
- new net: C28.1, U6.6 (BST)
- new net LED_DIN: LED1.1 (DIN)
Other:
- note added: "5V DC-DC Converter (compact 2A max Version)"

Commit message: Schematic Updates Madrilla
Parts:
- removed U9: TPS54202DDC, Package_TO_SOT_SMD:SOT-23-6, symbol Regulator_Switching:TPS54202DDC
- L3: LCSC C436530 -> C167874
Connections:
- no-connect marks 7 -> 8
Other:
- note added: "Caps could be added to filter input voltage, but we should already have sufficient bulk filtering close by"
- note added: "Side Facing Adressable LEDs (used for Iluminating the Z Probe during leveling)"
- moved on the sheet: C11, C12, C14, C16, C18, C20, C27, C28, C30, C31, C5, C7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

Commit message: update to Kicad 9.0.X
Parts:
- L3: footprint Vortac:L_Sunlord_MWSA0518_5.4x5.2mm -> Vortac:IND-SMD_L4.0-W4.0_FNR40XXS
Changed lines of the file:
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@@
 (kicad_sch
-	(version 20231120)
+	(version 20250114)
 	(generator "eeschema")
-	(generator_version "8.0")
+	(generator_version "9.0")
 	(paper "A4")
 	(title_block
@@
 		(comment 4 "-- VORTAC PCB --")
 	)
+	(rectangle
+		(start 16.51 130.81)
+		(end 83.82 193.04)
+		(stroke
+			(width 0)
+			(type dash)
+		)
+		(fill
+			(type none)
+		)
+	)
+	(rectangle
+		(start 143.51 16.51)
+		(end 280.67 74.93)
+		(stroke
+			(width 0)
+			(type dash)
+		)
+		(fill
+			(type none)
+		)
+	)
+	(rectangle
+		(start 16.51 16.51)
+		(end 139.7 74.93)
+		(stroke
+			(width 0)
+			(type dash)
+		)
+		(fill
+			(type none)
+		)
+	)
+	(rectangle
+		(start 88.9 166.37)
+		(end 139.7 193.04)
+		(stroke
+			(width 0)
+			(type dash)
+		)
+		(fill
+			(type none)
+		)
+	)
+	(text "Magnetic Angle Sensor\n(IC using two internal hall sensors)"
+		(exclude_from_sim no)
+		(at 21.844 140.462 0)
+		(effects
+			(font
+				(size 1.8034 1.8034)
+			)
+			(justify left bottom)
+		)
+	)
+	(text "R2 = 0.8 / (VOUT-0.8) * 100K\nR2 = 19.047 >> 19.1K\n\nVOUT = 0.8 * R1/R2 + 0.8\nVOUT = 4.98V\n\nRT = 55300/FSW^-1.025\nRT(500 kHz) = 94.68K"
+		(exclude_from_sim no)
+		(at -105.41 123.19 0)
+		(effects
+			(font
+				(size 1.27 1.27)
+			)
+			(justify left bottom)
+		)
+	)
+	(text "5V DC-DC Converter\n(capable of min 2.5A)"
+		(exclude_from_sim no)
+		(at -110.998 88.138 0)
+		(effects
+			(font
+				(size 1.8034 1.8034)
+			)
+			(justify left bottom)
+		)
+	)
+	(text "Side Facing Adressable LEDs\n(used for Iluminating the Z Probe during leveling)"
+		(exclude_from_sim no)
+		(at 150.368 27.178 0)
+		(effects
+			(font
+				(size 1.8034 1.8034)
+			)
+			(justify left bottom)
+		)
+	)
+	(text "Optical Endstops\n(endstop doubles as bed prope)"
+		(exclude_from_sim no)
+		(at 21.336 25.908 0)
+		(effects
+			(font
+				(size 1.8034 1.8034)
+			)
+			(justify left bottom)
+		)
+	)
+	(text "TOOL ID\n(sense pin)"
+		(exclude_from_sim no)
+		(at 92.964 175.006 0)
+		(effects
+			(font
+				(size 1.8034 1.8034)
+			)
+			(justify left bottom)
+		)
+	)
+	(text "3.3V Linear Voltage Regulator\n(300mA for internal use only)"
+		(exclude_from_sim no)
+		(at 91.44 139.7 0)
+		(effects
+			(font
+				(size 1.8034 1.8034)
+			)
+			(justify left bottom)
+		)
+	)
+	(text "Caps could be added to filter input voltage, \nbut we should already have sufficient bulk filtering close by"
+		(exclude_from_sim no)
+		(at 151.892 64.77 0)
+		(effects
+			(font
+				(size 0.7874 0.7874)
+			)
+			(justify left top)
+		)
+	)
+	(text "5V DC-DC Converter\n(compact 2A max Version)"
+		(exclude_from_sim no)
+		(at 20.828 87.63 0)
+		(effects
+			(font
+				(size 1.8034 1.8034)
+			)
+			(justify left bottom)
+		)
+	)
 	(junction
 		(at -39.37 118.11)
@@
 		)
 	)
-	(rectangle
-		(start 16.51 130.81)
-		(end 83.82 193.04)
-		(stroke
-			(width 0)
-			(type dash)
-		)
-		(fill
-			(type none)
-		)
-	)
-	(rectangle
-		(start 143.51 16.51)
-		(end 280.67 74.93)
-		(stroke
-			(width 0)
-			(type dash)
-		)
-		(fill
-			(type none)
-		)
-	)
-	(rectangle
-		(start 16.51 16.51)
-		(end 139.7 74.93)
-		(stroke
-			(width 0)
-			(type dash)
-		)
-		(fill
-			(type none)
-		)
-	)
-	(rectangle
-		(start 88.9 166.37)
-		(end 139.7 193.04)
-		(stroke
-			(width 0)
-			(type dash)
-		)
-		(fill
-			(type none)
-		)
-	)
-	(text "Magnetic Angle Sensor\n(IC using two internal hall sensors)"
-		(exclude_from_sim no)
-		(at 21.844 140.462 0)
-		(effects
-			(font
-				(size 1.8034 1.8034)
-			)
-			(justify left bottom)
-		)
-	)
-	(text "R2 = 0.8 / (VOUT-0.8) * 100K\nR2 = 19.047 >> 19.1K\n\nVOUT = 0.8 * R1/R2 + 0.8\nVOUT = 4.98V\n\nRT = 55300/FSW^-1.025\nRT(500 kHz) = 94.68K"
-		(exclude_from_sim no)
-		(at -105.41 123.19 0)
-		(effects
-			(font
-				(size 1.27 1.27)
-			)
-			(justify left bottom)
-		)
-	)
-	(text "5V DC-DC Converter\n(capable of min 2.5A)"
-		(exclude_from_sim no)
-		(at -110.998 88.138 0)
-		(effects
-			(font
-				(size 1.8034 1.8034)
-			)
-			(justify left bottom)
-		)
-	)
-	(text "Side Facing Adressable LEDs\n(used for Iluminating the Z Probe during leveling)"
-		(exclude_from_sim no)
-		(at 150.368 27.178 0)
-		(effects
-			(font
-				(size 1.8034 1.8034)
-			)
-			(justify left bottom)
-		)
-	)
-	(text "Optical Endstops\n(endstop doubles as bed prope)"
-		(exclude_from_sim no)
-		(at 21.336 25.908 0)
-		(effects
-			(font
-				(size 1.8034 1.8034)
-			)
-			(justify left bottom)
-		)
-	)
-	(text "TOOL ID\n(sense pin)"
-		(exclude_from_sim no)
-		(at 92.964 175.006 0)
-		(effects
-			(font
-				(size 1.8034 1.8034)
-			)
-			(justify left bottom)
-		)
-	)
-	(text "3.3V Linear Voltage Regulator\n(300mA for internal use only)"
-		(exclude_from_sim no)
-		(at 91.44 139.7 0)
-		(effects
-			(font
-				(size 1.8034 1.8034)
-			)
-			(justify left bottom)
-		)
-	)
-	(text "Caps could be added to filter input voltage, \nbut we should already have sufficient bulk filtering close by"
-		(exclude_from_sim no)
-		(at 151.892 64.77 0)
-		(effects
-			(font
-				(size 0.7874 0.7874)
-			)
-			(justify left top)
-		)
-	)
-	(text "5V DC-DC Converter\n(compact 2A max Version)"
-		(exclude_from_sim no)
-		(at 20.828 87.63 0)
-		(effects
-			(font
-				(size 1.8034 1.8034)
-			)
-			(justify left bottom)
-		)
-	)
 	(global_label "AS_MISO"
 		(shape input)
@@
 			)
 		)
-		(property "Footprint" "Vortac:L_Sunlord_MWSA0518_5.4x5.2mm"
+		(property "Footprint" "Vortac:IND-SMD_L4.0-W4.0_FNR40XXS"
 			(at 91.44 99.06 0)
 			(effects

Commit message: pushy
Parts:
- removed C11, C7: 0.1uF 50V, Capacitor_SMD:C_0603_1608Metric, symbol Device:C_Small
- removed C12: 3.3nF, Capacitor_SMD:C_0603_1608Metric, symbol Device:C_Small
- removed C14: 56pF, Capacitor_SMD:C_0603_1608Metric, symbol Device:C_Small
- removed C16, C18, C20: 47uF, Capacitor_SMD:C_0805_2012Metric, symbol Device:C_Small
- removed C49: 0.1uF 16V, Capacitor_SMD:C_0402_1005Metric, symbol Device:C_Small
- removed C5: 10uF 50V, Capacitor_SMD:C_1206_3216Metric, symbol Device:C_Small
- removed L2: 10uH, Vortac:L_Sunlord_MWSA0518_5.4x5.2mm, symbol Device:L
- removed R23: 10k, Resistor_SMD:R_0402_1005Metric, symbol Device:R_Small
- removed R25: 95k, Resistor_SMD:R_0402_1005Metric, symbol Device:R_Small
- removed R28: 100k, Resistor_SMD:R_0402_1005Metric, symbol Device:R_Small
- removed R29: 19.1k, Resistor_SMD:R_0402_1005Metric, symbol Device:R_Small
- removed R51: 1K, Resistor_SMD:R_0402_1005Metric, symbol Device:R_Small
- removed R52: 10K, Resistor_SMD:R_0402_1005Metric, symbol Device:R_Small
- removed U4: TPS54335ADRCR, Vortac:VSON-10-1EP_3x3mm_P0.5mm_EP1.65x2.4mm_ThermalVias, symbol ToolChanger:TPS54335ADRCR
Connections:
- no-connect marks 8 -> 7
Other:
- note removed: "5V DC-DC Converter (capable of min 2.5A)"
- note removed: "R2 = 0.8 / (VOUT-0.8) * 100K R2 = 19.047 >> 19.1K VOUT = 0.8 * R1/R2 + 0.8 VOUT = 4.98V RT = 55300/FSW^-1.025 RT(500 kHz) = 94.68K"
- note removed: "TOOL ID (sense pin)"

Commit message: Update Symbol Librarys
Parts:
- U7: symbol VORTAC_REV1-rescue:EE-SX3350 -> Vortac:EE-SX3350

Commit message: updated revs fabrication test
Parts:
- U3: LCSC EE-SX4320 -> C469129
Changed lines of the file:
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@@
 			)
 		)
-		(property "LCSC" "EE-SX4320"
+		(property "LCSC" "C469129"
 			(at 52.07 34.29 0)
 			(effects

Commit message: night night
Parts:
- added Q3: BSS138AKDW, Package_TO_SOT_SMD:SOT-363_SC-70-6, symbol Vortac:BSS138AKDW
- added R16: 10K, Resistor_SMD:R_0402_1005Metric, symbol Device:R_Small
Connections:
- net +3V3: now also R16.1
- new net: Q3.1 (S1), Q3.4 (S2)
- new net CAN_TRM: Q3.2 (G1), Q3.5 (G2), R16.2
- new net CAN_TRM_H: Q3.6 (D1)
- new net CAN_TRM_L: Q3.3 (D2)
Other:
- note added: "Controllable CAN Terminator"
- moved on the sheet: C15, C27, C28, C3, C30, C31, C8, L3, R14, U1, U5, U6

Commit message: Anned Parts
Parts:
- C15, C28: footprint Capacitor_SMD:C_0603_1608Metric -> Capacitor_SMD:C_0402_1005Metric; LCSC C1591 -> C5182432
- C19, C25: value 0.1uF 16V -> 0.1uF 50V; LCSC C1525 -> C5182432
- C27: footprint Capacitor_SMD:C_1206_3216Metric -> Capacitor_SMD:C_0805_2012Metric; LCSC C89632 -> C440198
- C3, C8: value 1uF -> 1uF 16V; LCSC (none) -> C106248; description (none) -> could be 0.1 to 1uf
- C30, C31: value 22uF -> 22uF 16V; LCSC C466799 -> C2762594; description (none) -> could be 10V maybe 0402
- LED1, LED2: LCSC (none) -> C2890037; LCSC Part C2890037 -> (none)
- Q3: LCSC (none) -> C5224287; LCSC Part C5224287 -> (none)
- R1, R15: LCSC (none) -> C106235
- R14, R16, R2, R8: LCSC (none) -> C60490
- R5, R6: footprint Resistor_SMD:R_0603_1608Metric -> Resistor_SMD:R_0402_1005Metric; LCSC (none) -> C6117577
