File: PCB/VORTAC/KiCAD/VORTAC_REV1/Logic.kicad_sch (KiCad schematic)
At the start: 26 parts, among them Q3 BSS138AKDW, U1 TLV73333PDBV, U3 EE-SX4320, U5 AS5047D, U6 AP63205WU, U7 EE-SX3350

Commit message: Evil Mita is v00:98
Parts:
- C3, C8: description could be 0.1 to 1uf -> (none); notes (none) -> could be 0.1 to 1uf
- C30, C31: description could be 10V maybe 0402 -> (none); notes (none) -> could be 10V maybe 0402

Commit message: No Body knows.... The trouble I've seen
Other:
- moved on the sheet: C31
Changed lines of the file:
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@@
 	)
 	(junction
-		(at 109.22 97.79)
+		(at 114.3 97.79)
 		(diameter 0)
 		(color 0 0 0 0)
@@
 	(wire
 		(pts
-			(xy 100.33 97.79) (xy 109.22 97.79)
+			(xy 100.33 97.79) (xy 114.3 97.79)
 		)
 		(stroke
@@
 	(wire
 		(pts
-			(xy 109.22 97.79) (xy 116.84 97.79)
-		)
-		(stroke
-			(width 0)
-			(type default)
-		)
-	)
-	(wire
-		(pts
 			(xy 35.56 162.56) (xy 39.37 162.56)
 		)
@@
 	(wire
 		(pts
-			(xy 109.22 97.79) (xy 109.22 100.33)
+			(xy 114.3 97.79) (xy 114.3 100.33)
 		)
 		(stroke
@@
 	(wire
 		(pts
-			(xy 109.22 105.41) (xy 109.22 107.95)
+			(xy 114.3 105.41) (xy 114.3 107.95)
 		)
 		(stroke
@@
 	(wire
 		(pts
-			(xy 109.22 107.95) (xy 100.33 107.95)
+			(xy 114.3 107.95) (xy 100.33 107.95)
 		)
 		(stroke
@@
 	(wire
 		(pts
+			(xy 114.3 97.79) (xy 119.38 97.79)
+		)
+		(stroke
+			(width 0)
+			(type default)
+		)
+	)
+	(wire
+		(pts
 			(xy 92.71 62.23) (xy 105.41 62.23)
 		)
@@
 	(symbol
 		(lib_id "power:+5V")
-		(at 116.84 97.79 270)
+		(at 119.38 97.79 270)
 		(unit 1)
 		(exclude_from_sim no)
@@
 		(dnp no)
 		(property "Reference" "#PWR37"
-			(at 113.03 97.79 0)
+			(at 115.57 97.79 0)
 			(effects
 				(font
@@
 		)
 		(property "Value" "+5V"
-			(at 120.0912 98.171 90)
+			(at 122.6312 98.171 90)
 			(effects
 				(font
@@
 		)
 		(property "Footprint" ""
-			(at 116.84 97.79 0)
+			(at 119.38 97.79 0)
 			(effects
 				(font
@@
 		)
 		(property "Datasheet" ""
-			(at 116.84 97.79 0)
+			(at 119.38 97.79 0)
 			(effects
 				(font
@@
 		)
 		(property "Description" "Power symbol creates a global label with name \"+5V\""
-			(at 116.84 97.79 0)
+			(at 119.38 97.79 0)
 			(effects
 				(font
@@
 		)
 		(property "Value" "22uF 16V"
-			(at 104.902 92.202 0)
+			(at 107.188 101.092 0)
 			(effects
 				(font
@@
 	(symbol
 		(lib_id "Device:C_Small")
-		(at 109.22 102.87 0)
+		(at 114.3 102.87 0)
 		(unit 1)
 		(exclude_from_sim no)
@@
 		(dnp no)
 		(property "Reference" "C31"
-			(at 113.03 104.14 0)
+			(at 118.11 104.14 0)
 			(effects
 				(font
@@
 		)
 		(property "Value" "22uF 16V"
-			(at 113.03 101.6 0)
+			(at 121.412 101.092 0)
 			(effects
 				(font
@@
 		)
 		(property "Footprint" "Capacitor_SMD:C_0805_2012Metric"
-			(at 109.22 102.87 0)
+			(at 114.3 102.87 0)
 			(effects
 				(font
@@
 		)
 		(property "Datasheet" "~"
-			(at 109.22 102.87 0)
+			(at 114.3 102.87 0)
 			(effects
 				(font
@@
 		)
 		(property "Description" "Unpolarized capacitor, small symbol"
-			(at 109.22 102.87 0)
+			(at 114.3 102.87 0)
 			(effects
 				(font
@@
 		)
 		(property "LCSC" "C2762594"
-			(at 109.22 102.87 0)
+			(at 114.3 102.87 0)
 			(effects
 				(font
@@
 		)
 		(property "notes" "could be 10V maybe 0402"
-			(at 109.22 102.87 0)
+			(at 114.3 102.87 0)
 			(effects
 				(font

Commit message: Girl Math
Parts:
- C30, C31: footprint Capacitor_SMD:C_0805_2012Metric -> Capacitor_SMD:C_0603_1608Metric
Connections:
- net CAN_TRM_H: now also Q3.3 (D2); no longer Q3.6 (D1)
- net CAN_TRM_L: now also Q3.6 (D1); no longer Q3.3 (D2)
Changed lines of the file:
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@@
 	(global_label "CAN_TRM_H"
 		(shape input)
-		(at 123.19 176.53 0)
+		(at 102.87 181.61 180)
 		(effects
 			(font
 				(size 1.27 1.27)
 			)
-			(justify left)
+			(justify right)
 		)
 		(property "Intersheetrefs" "${INTERSHEET_REFS}"
-			(at 123.19 176.53 0)
+			(at 102.87 181.61 0)
 			(effects
 				(font
@@
 	(global_label "CAN_TRM_L"
 		(shape input)
-		(at 102.87 181.61 180)
+		(at 123.19 176.53 0)
 		(effects
 			(font
 				(size 1.27 1.27)
 			)
-			(justify right)
+			(justify left)
 		)
 		(property "Intersheetrefs" "${INTERSHEET_REFS}"
-			(at 102.87 181.61 0)
+			(at 123.19 176.53 0)
 			(effects
 				(font
@@
 			)
 		)
-		(property "Footprint" "Capacitor_SMD:C_0805_2012Metric"
+		(property "Footprint" "Capacitor_SMD:C_0603_1608Metric"
 			(at 100.33 102.87 0)
 			(effects
@@
 			)
 		)
-		(property "Footprint" "Capacitor_SMD:C_0805_2012Metric"
+		(property "Footprint" "Capacitor_SMD:C_0603_1608Metric"
 			(at 114.3 102.87 0)
 			(effects

Commit message: Route me like one of you French girls
Parts:
- removed Q3: BSS138AKDW, Package_TO_SOT_SMD:SOT-363_SC-70-6, symbol Vortac:BSS138AKDW
- removed R16: 10K, Resistor_SMD:R_0402_1005Metric, symbol Device:R_Small
Other:
- note removed: "Controllable CAN Terminator"

Commit message: I NEED A HEEEROOO
Connections:
- net +5V_OUT: now reaches C28.2, L3.1, U6.5 (SW)
- net +5V_BST: now reaches C28.1, U6.6 (BST)
Other:
- moved on the sheet: C27, C28, C30, C31, L3, U6

Commit message: KONGSTRONG
Parts:
- U7: value EE-SX3350 -> EE-SX4350; LCSC C7470740 -> C17524058
Changed lines of the file:
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@@
 			)
 		)
-		(property "Value" "EE-SX3350"
+		(property "Value" "EE-SX4350"
 			(at 72.39 52.07 0)
 			(effects
@@
 			)
 		)
-		(property "LCSC" "C7470740"
+		(property "LCSC" "C17524058"
 			(at 52.07 57.15 0)
 			(effects
