File: PCB/VORTAC/KiCAD/VORTAC_TOOLPLATE_REV1/VORTAC_TOOLPLATE_REV1/VORTAC_TOOLPLATE_REV1.kicad_pcb (KiCad board)
At the start: 4 copper layers, 15.4 x 19.5 mm, 6 parts, among them J1 Conn_01x07, J2 Conn_01x02

Commit message: MEIN BEEEEEIIIINNNN
Parts:
- added J3: Conn_01x05, Vortac:Toolplate_Solderpoint_01x05_Data, F.Cu at (121.1, 75.8)
- moved H2 7.81 mm to (117.7, 88.0)
- moved D2 1.18 mm to (116.7, 79.6)
- moved D1 0.55 mm to (116.7, 83.2)
- moved J2 0.20 mm to (120.3, 69.0)
Connections:
- J2 pad 1: (no net) -> unconnected-(J2-Pin_1-Pad1)
Other:
- board size 15.4 x 19.5 mm -> 15.4 x 24 mm

Commit message: Churro
Parts:
- moved D2 5.77 mm to (116.3, 73.8)
- moved D1 0.50 mm to (116.4, 83.6)
- moved J2 0.06 mm to (120.3, 69.0)
Connections:
- J1 pad 3: GND -> VDC
- J1 pad 4: VDC -> TOOL_ID
- J1 pad 5: TOOL_ID -> GND
- J2 pad 1: unconnected-(J2-Pin_1-Pad1) -> GND
- J2 pad 2: unconnected-(J2-Pin_2-Pad2) -> VDC
- J3 pad 1: unconnected-(J3-Pin_1-Pad1) -> USB_90_D+
- J3 pad 2: unconnected-(J3-Pin_2-Pad2) -> USB_90_D-
- J3 pad 3: unconnected-(J3-Pin_3-Pad3) -> TOOL_ID
- J3 pad 4: unconnected-(J3-Pin_4-Pad4) -> CAN_H
- J3 pad 5: unconnected-(J3-Pin_5-Pad5) -> CAN_L
Routing:
- net USB_90_D-: track 0.00 -> 13.0 mm
- net TOOL_ID: track 0.00 -> 11.7 mm
- net CAN_H: track 0.00 -> 11.4 mm
- net USB_90_D+: track 0.00 -> 9.80 mm
- net CAN_L: track 0.00 -> 9.52 mm
- added copper zone on B.Cu, net GND
- added copper zone on F.Cu, net GND
- added copper zone on In1.Cu, net GND
- added copper zone on In2.Cu, net VDC

Commit message: KONGSTRONG
Parts:
- added D3: SD05, Diode_SMD:D_SOD-323, F.Cu at (118.4, 78.2)
- added D4: SD05, Diode_SMD:D_SOD-323, F.Cu at (118.4, 80.1)
- added D9: PTVS26VS1UR,115-ES, Diode_SMD:D_SOD-123F, F.Cu at (117.3, 74.2)
- D1, D2: value SP0502BAHT -> UDD32C24L01; footprint Package_TO_SOT_SMD:SOT-23 -> Diode_SMD:D_SOD-323
- moved D2 10.8 mm to (118.4, 84.5)
- moved D1 2.25 mm to (118.4, 82.6)
Connections:
- D1 pad 1: unconnected-(D1-K-Pad1) -> GND
- D1 pad 2: unconnected-(D1-K-Pad2) -> CAN_H
- D2 pad 1: unconnected-(D2-K-Pad1) -> GND
- D2 pad 2: unconnected-(D2-K-Pad2) -> CAN_L
- J3 pad 1: USB_90_D+ -> TOOL_ID
- J3 pad 2: USB_90_D- -> USB_90_D+
- J3 pad 3: TOOL_ID -> USB_90_D-
Routing:
- net USB_90_D+: track 9.80 -> 14.7 mm
- net VDC: track 0.00 -> 3.05 mm
- net CAN_L: track 9.52 -> 11.5 mm
- net USB_90_D-: track 13.0 -> 14.9 mm
- net GND: vias 0 -> 21
Other:
- board text added: "CH"
- board text added: "CL"
- board text added: "DM"
- board text added: "DP"
- board text added: "ID"
- board text added: "V+"
