File: PCB/VORTAC/KiCAD/VORTAC_TOOLPLATE_REV1/VORTAC_TOOLPLATE_REV1/VORTAC_TOOLPLATE_REV1.kicad_sch (KiCad schematic)
At the start: 6 parts, among them J1 Conn_01x07, J2 Conn_01x02

Commit message: MEIN BEEEEEIIIINNNN
Parts:
- added J3: Conn_01x05, Vortac:Toolplate_Solderpoint_01x05_Data, symbol Connector_Generic:Conn_01x05
Changed lines of the file:
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@@
+	)
+	(symbol
+		(lib_id "Connector_Generic:Conn_01x05")
+		(at 71.12 106.68 0)
+		(unit 1)
+		(exclude_from_sim no)
+		(in_bom yes)
+		(on_board yes)
+		(dnp no)
+		(property "Reference" "J3"
+			(at 69.85 117.856 0)
+			(effects
+				(font
+					(size 1.27 1.27)
+				)
+				(justify left)
+			)
+		)
+		(property "Value" "Conn_01x05"
+			(at 65.024 115.062 0)
+			(effects
+				(font
+					(size 1.27 1.27)
+				)
+				(justify left)
+			)
+		)
+		(property "Footprint" "Vortac:Toolplate_Solderpoint_01x05_Data"
+			(at 71.12 118.618 0)
+			(effects
+				(font
+					(size 1.27 1.27)
+				)
+				(hide yes)
+			)
+		)
+		(property "Datasheet" "~"
+			(at 71.12 106.68 0)
+			(effects
+				(font
+					(size 1.27 1.27)
+				)
+				(hide yes)
+			)
+		)
+		(property "Description" "Generic connector, single row, 01x05, script generated (kicad-library-utils/schlib/autogen/connector/)"
+			(at 71.12 106.68 0)
+			(effects
+				(font
+					(size 1.27 1.27)
+				)
+				(hide yes)
+			)
+		)
+		(pin "4"
+		)
+		(pin "3"
+		)
+		(pin "1"
+		)
+		(pin "2"
+		)
+		(pin "5"
+		)
+		(instances
+			(project ""
+				(path "/b23b3086-82ed-4285-9d49-d03b4e41a1a0"
+					(reference "J3")
+					(unit 1)
+				)
+			)
+		)
 	)
 	(symbol

Commit message: Churro
Connections:
- net CAN_H: now also J3.4 (Pin_4)
- net CAN_L: now also J3.5 (Pin_5)
- net GND: now also J1.5 (Pin_5), J2.1 (Pin_1); no longer J1.3 (Pin_3)
- net TOOL_ID: now also J1.4 (Pin_4), J3.3 (Pin_3); no longer J1.5 (Pin_5)
- net USB_90_D+: now also J3.1 (Pin_1)
- net USB_90_D-: now also J3.2 (Pin_2)
- net VDC: now also J1.3 (Pin_3), J2.2 (Pin_2); no longer J1.4 (Pin_4)
Other:
- note added: "Grabber Connection"
- note added: "Tool Wire Harness"
- note removed: "Tool Connection"
- moved on the sheet: J2, J3

Commit message: KONGSTRONG
Parts:
- removed D1, D2: SP0502BAHT, Package_TO_SOT_SMD:SOT-23, symbol Power_Protection:SP0502BAHT
- added D1, D2: UDD32C24L01, Diode_SMD:D_SOD-323, symbol Diode:SD24_SOD323
- added D3, D4: SD05, Diode_SMD:D_SOD-323, symbol Diode:SD24_SOD323
- added D9: PTVS26VS1UR,115-ES, Diode_SMD:D_SOD-123F, symbol Diode:SD24_SOD323
Connections:
- net CAN_H: now also D1.2 (A2)
- net CAN_L: now also D2.2 (A2)
- net GND: now also D1.1 (A1), D2.1 (A1), D3.1 (A1), D4.1 (A1), D9.1 (A1)
- net TOOL_ID: now also J3.1 (Pin_1); no longer J3.3 (Pin_3)
- net USB_90_D+: now also J3.2 (Pin_2), D3.2 (A2); no longer J3.1 (Pin_1)
- net USB_90_D-: now also J3.3 (Pin_3), D4.2 (A2); no longer J3.2 (Pin_2)
- net VDC: now also D9.2 (A2)
Other:
- note added: "ESD TVS Diodes CAN"
- note added: "ESD TVS Diodes USB"
