File: PCB/VORTAC/KiCAD/VORTAC_FRONT_REV1/VORTAC_FRONT_REV1.kicad_pcb (KiCad board)
At the start: 4 copper layers, 31.9 x 51.5 mm, 5 parts, among them J1 Conn_02x02_Odd_Even, J2 Conn_02x03_Odd_Even, J3 Conn_01x07

Commit message: No Body knows.... The trouble I've seen
Parts:
- moved J1 3.91 mm to (122.7, 101.4), turned to 45 degrees
- moved H1 0.19 mm to (124.4, 105.0)
Connections:
- J1 pad 1: VDC -> TOOL_ID
- J1 pad 2: CAN_H -> CAN_L
- J1 pad 3: CAN_L -> VDC
- J1 pad 4: TOOL_ID -> CAN_H
- J2 pad 1: VDC -> CAN_L
- J2 pad 3: CAN_L -> USB_D+
- J2 pad 5: USB_D+ -> VDC
- J3 pad 1: CAN_H -> USB_D+
- J3 pad 2: CAN_L -> USB_D-
- J3 pad 6: USB_D+ -> CAN_H
- J3 pad 7: USB_D- -> CAN_L
Routing:
- net CAN_L: track 0.00 -> 37.8 mm
- net CAN_H: track 0.00 -> 34.8 mm
- net USB_D-: track 0.00 -> 20.5 mm
- net USB_D+: track 0.00 -> 17.2 mm
Other:
- board size 31.9 x 51.5 mm -> 31.7 x 51.3 mm

Commit message: FML
Parts:
- added NT1: NetTie_2, NetTie:NetTie-2_SMD_Pad0.5mm, F.Cu at (112.9, 79.3)
- H1, H2: footprint MountingHole:MountingHole_2.2mm_M2_Pad_Via -> Vortac:MountingHole_2.2mm_M2_Pad_Via_NTR
Connections:
- H1 pad 1: unconnected-(H1-Pad1) -> GND
- H2 pad 1: unconnected-(H2-Pad1) -> GND
- J1 pad 1: TOOL_ID -> GND
- J1 pad 2: CAN_L -> VDC
- J1 pad 3: VDC -> CAN_H
- J1 pad 4: CAN_H -> CAN_L
- J2 pad 2: TOOL_ID -> GND
- J3 pad 3: TOOL_ID -> GND
- J3 pad 6: CAN_H -> CAN_L
- J3 pad 7: CAN_L -> CAN_H
Routing:
- net CAN_H: track 34.8 -> 54.5 mm
- net USB_D-: track 20.5 -> 3.62 mm
- net CAN_L: track 37.8 -> 50.1 mm
- net GND: vias 0 -> 31
- added copper zone on B.Cu, net GND
- added copper zone on F.Cu, net GND
- added copper zone on In1.Cu, net GND
- added copper zone on In2.Cu, net VDC

Commit message: USB C Survivor
Changed lines of the file:
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@@
 		(start 110.1 74.6)
 		(end 108.13 74.6)
-		(width 0.2)
+		(width 0.3)
 		(layer "F.Cu")
 		(net 5)
@@
 		(start 108.13 74.6)
 		(end 106.96 73.43)
-		(width 0.2)
+		(width 0.3)
 		(layer "F.Cu")
 		(net 5)
@@
 		(start 108.867146 72.867146)
 		(end 112.026746 72.867146)
-		(width 0.2)
+		(width 0.3)
 		(layer "F.Cu")
 		(net 6)
@@
 		(start 110.75 62.65)
 		(end 106.4 67)
-		(width 0.2)
+		(width 0.3)
 		(layer "F.Cu")
 		(net 6)
@@
 		(start 106.4 70.4)
 		(end 108.867146 72.867146)
-		(width 0.2)
+		(width 0.3)
 		(layer "F.Cu")
 		(net 6)
@@
 		(start 110.75 61.7)
 		(end 110.75 62.65)
-		(width 0.2)
+		(width 0.3)
 		(layer "F.Cu")
 		(net 6)
@@
 		(start 106.4 67)
 		(end 106.4 70.4)
-		(width 0.2)
+		(width 0.3)
 		(layer "F.Cu")
 		(net 6)

Commit message: Churro
Parts:
- moved NT1 1.82 mm to (111.1, 79.4), turned to -38 degrees
Connections:
- J2 pad 1: CAN_L -> CAN_H
- J2 pad 4: CAN_H -> CAN_L
- J3 pad 3: GND -> VDC
- J3 pad 4: VDC -> TOOL_ID
- J3 pad 5: TOOL_ID -> GND
Routing:
- net USB_D-: track 3.62 -> 20.5 mm
- net CAN_L: track 50.1 -> 60.9 mm
- net CAN_H: track 54.5 -> 61.2 mm
- net USB_D+: track 17.2 -> 18.1 mm

Commit message: KONGSTRONG
Connections:
- J2 pad 2: GND -> VDC
- J2 pad 5: VDC -> GND

Commit message: Yippiieeeee
Parts:
- moved NT1 0.14 mm to (111.2, 79.4)
Routing:
- net VDC: track 0.00 -> 5.11 mm, vias 0 -> 3
- net USB_D+: track 18.1 -> 22.6 mm
- net USB_D-: track 20.5 -> 21.6 mm
- net GND: vias 31 -> 63
Other:
- board text added: "VORTAC"
