File: PCB/VORTAC/KiCAD/VORTAC_FRONT_REV1/VORTAC_FRONT_REV1.kicad_pcb (KiCad board)
At the start: 4 copper layers, 31.7 x 51.3 mm, 6 parts, among them J1 Conn_02x02_Odd_Even, J2 Conn_02x03_Odd_Even, J3 Conn_01x07

Commit message: idk
Other:
- board text removed: "VORTAC"
