File: PCB/VORTAC/KiCAD/VORTAC_FRONT_REV1/VORTAC_FRONT_REV1.kicad_sch (KiCad schematic)
At the start: 5 parts, among them J1 Conn_02x02_Odd_Even, J2 Conn_02x03_Odd_Even, J3 Conn_01x07

Commit message: No Body knows.... The trouble I've seen
Connections:
- net CAN_H: now also J1.4 (Pin_4), J3.6 (Pin_6); no longer J1.2 (Pin_2), J3.1 (Pin_1)
- net CAN_L: now also J1.2 (Pin_2), J2.1 (Pin_1), J3.7 (Pin_7); no longer J1.3 (Pin_3), J2.3 (Pin_3), J3.2 (Pin_2)
- net GND: now also J1.1 (Pin_1); no longer J1.4 (Pin_4)
- net USB_D+: now also J2.3 (Pin_3), J3.1 (Pin_1); no longer J2.5 (Pin_5), J3.6 (Pin_6)
- net USB_D-: now also J3.2 (Pin_2); no longer J3.7 (Pin_7)
- net VDC: now also J1.3 (Pin_3), J2.5 (Pin_5); no longer J1.1 (Pin_1), J2.1 (Pin_1)

Commit message: FML
Parts:
- added NT1: NetTie_2, NetTie:NetTie-2_SMD_Pad0.5mm, symbol Device:NetTie_2
- H1, H2: footprint MountingHole:MountingHole_2.2mm_M2_Pad_Via -> Vortac:MountingHole_2.2mm_M2_Pad_Via_NTR
- J1: LCSC (none) -> C2840016
- J2: LCSC (none) -> C234188
Connections:
- net CAN_H: now also J1.3 (Pin_3), J3.7 (Pin_7); no longer J1.4 (Pin_4), J3.6 (Pin_6)
- net CAN_L: now also J1.4 (Pin_4), J3.6 (Pin_6); no longer J1.2 (Pin_2), J3.7 (Pin_7)
- net GND: now also H1.1, H2.1, NT1.2; no longer J3.5 (Pin_5)
- net VDC: now also J1.2 (Pin_2); no longer J1.3 (Pin_3)
- new net TOOL_ID: J3.5 (Pin_5), NT1.1
Other:
- note added: "Mounting Holes"
- moved on the sheet: H1, H2

Commit message: Churro
Connections:
- net CAN_H: now also J2.1 (Pin_1); no longer J2.4 (Pin_4)
- net CAN_L: now also J2.4 (Pin_4); no longer J2.1 (Pin_1)
- net GND: now also J3.5 (Pin_5); no longer J3.3 (Pin_3)
- net TOOL_ID: now also J3.4 (Pin_4); no longer J3.5 (Pin_5)
- net VDC: now also J3.3 (Pin_3); no longer J3.4 (Pin_4)
Changed lines of the file:
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@@
 	(global_label "CAN_H"
 		(shape input)
-		(at 64.77 86.36 0)
+		(at 44.45 83.82 180)
 		(fields_autoplaced yes)
 		(effects
@@
 				(size 1.27 1.27)
 			)
-			(justify left)
+			(justify right)
 		)
 		(property "Intersheetrefs" "${INTERSHEET_REFS}"
-			(at 73.7424 86.36 0)
-			(effects
-				(font
-					(size 1.27 1.27)
-				)
-				(justify left)
+			(at 35.4776 83.82 0)
+			(effects
+				(font
+					(size 1.27 1.27)
+				)
+				(justify right)
 				(hide yes)
 			)
@@
 	(global_label "TOOL_ID"
 		(shape input)
-		(at 50.8 134.62 180)
+		(at 50.8 132.08 180)
 		(fields_autoplaced yes)
 		(effects
@@
 		)
 		(property "Intersheetrefs" "${INTERSHEET_REFS}"
-			(at 40.3157 134.62 0)
+			(at 40.3157 132.08 0)
 			(effects
 				(font
@@
 	(global_label "CAN_L"
 		(shape input)
-		(at 44.45 83.82 180)
+		(at 64.77 86.36 0)
 		(fields_autoplaced yes)
 		(effects
@@
 				(size 1.27 1.27)
 			)
-			(justify right)
+			(justify left)
 		)
 		(property "Intersheetrefs" "${INTERSHEET_REFS}"
-			(at 35.78 83.82 0)
-			(effects
-				(font
-					(size 1.27 1.27)
-				)
-				(justify right)
+			(at 73.44 86.36 0)
+			(effects
+				(font
+					(size 1.27 1.27)
+				)
+				(justify left)
 				(hide yes)
 			)
@@
 	(symbol
 		(lib_id "power:VDC")
-		(at 50.8 132.08 90)
+		(at 50.8 129.54 90)
 		(unit 1)
 		(exclude_from_sim no)
@@
 		(fields_autoplaced yes)
 		(property "Reference" "#PWR05"
-			(at 54.61 132.08 0)
+			(at 54.61 129.54 0)
 			(effects
 				(font
@@
 		)
 		(property "Value" "VDC"
-			(at 46.99 132.0801 90)
+			(at 46.99 129.5401 90)
 			(effects
 				(font
@@
 		)
 		(property "Footprint" ""
-			(at 50.8 132.08 0)
+			(at 50.8 129.54 0)
 			(effects
 				(font
@@
 		)
 		(property "Datasheet" ""
-			(at 50.8 132.08 0)
+			(at 50.8 129.54 0)
 			(effects
 				(font
@@
 		)
 		(property "Description" "Power symbol creates a global label with name \"VDC\""
-			(at 50.8 132.08 0)
+			(at 50.8 129.54 0)
 			(effects
 				(font
@@
 	(symbol
 		(lib_id "power:GND")
-		(at 50.8 129.54 270)
+		(at 50.8 134.62 270)
 		(unit 1)
 		(exclude_from_sim no)
@@
 		(fields_autoplaced yes)
 		(property "Reference" "#PWR06"
-			(at 44.45 129.54 0)
+			(at 44.45 134.62 0)
 			(effects
 				(font
@@
 		)
 		(property "Value" "GND"
-			(at 46.99 129.5401 90)
+			(at 46.99 134.6201 90)
 			(effects
 				(font
@@
 		)
 		(property "Footprint" ""
-			(at 50.8 129.54 0)
+			(at 50.8 134.62 0)
 			(effects
 				(font
@@
 		)
 		(property "Datasheet" ""
-			(at 50.8 129.54 0)
+			(at 50.8 134.62 0)
 			(effects
 				(font
@@
 		)
 		(property "Description" "Power symbol creates a global label with name \"GND\" , ground"
-			(at 50.8 129.54 0)
-			(effects
-				(font
+			(at 50.8 134.62 0)
+			(effects
+				(font

Commit message: KONGSTRONG
Connections:
- net GND: now also J2.5 (Pin_5); no longer J2.2 (Pin_2)
- net VDC: now also J2.2 (Pin_2); no longer J2.5 (Pin_5)
Changed lines of the file:
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@@
 		(on_board yes)
 		(dnp no)
-		(fields_autoplaced yes)
 		(property "Reference" "#PWR02"
 			(at 60.96 46.99 0)
@@
 	(symbol
 		(lib_id "power:GND")
-		(at 64.77 83.82 90)
+		(at 44.45 88.9 270)
 		(unit 1)
 		(exclude_from_sim no)
@@
 		(fields_autoplaced yes)
 		(property "Reference" "#PWR04"
-			(at 71.12 83.82 0)
+			(at 38.1 88.9 0)
 			(effects
 				(font
@@
 		)
 		(property "Value" "GND"
-			(at 68.58 83.8199 90)
+			(at 40.64 88.8999 90)
 			(effects
 				(font
@@
 		)
 		(property "Footprint" ""
-			(at 64.77 83.82 0)
-			(effects
-				(font
-					(size 1.27 1.27)
-				)
-				(hide yes)
-			)
-		)
-		(property "Datasheet" ""
-			(at 64.77 83.82 0)
+			(at 44.45 88.9 0)
+			(effects
+				(font
+					(size 1.27 1.27)
+				)
+				(hide yes)
+			)
+		)
+		(property "Datasheet" ""
+			(at 44.45 88.9 0)
 			(effects
 				(font
@@
 		)
 		(property "Description" "Power symbol creates a global label with name \"GND\" , ground"
-			(at 64.77 83.82 0)
+			(at 44.45 88.9 0)
 			(effects
 				(font
@@
 	(symbol
 		(lib_id "power:VDC")
-		(at 44.45 88.9 90)
+		(at 64.77 83.82 270)
 		(unit 1)
 		(exclude_from_sim no)
@@
 		(fields_autoplaced yes)
 		(property "Reference" "#PWR03"
-			(at 48.26 88.9 0)
+			(at 60.96 83.82 0)
 			(effects
 				(font
@@
 		)
 		(property "Value" "VDC"
-			(at 40.64 88.8999 90)
-			(effects
-				(font
-					(size 1.27 1.27)
-				)
-				(justify left)
-			)
-		)
-		(property "Footprint" ""
-			(at 44.45 88.9 0)
-			(effects
-				(font
-					(size 1.27 1.27)
-				)
-				(hide yes)
-			)
-		)
-		(property "Datasheet" ""
-			(at 44.45 88.9 0)
+			(at 68.58 83.8199 90)
+			(effects
+				(font
+					(size 1.27 1.27)
+				)
+				(justify left)
+			)
+		)
+		(property "Footprint" ""
+			(at 64.77 83.82 0)
+			(effects
+				(font
+					(size 1.27 1.27)
+				)
+				(hide yes)
+			)
+		)
+		(property "Datasheet" ""
+			(at 64.77 83.82 0)
 			(effects
 				(font
@@
 		)
 		(property "Description" "Power symbol creates a global label with name \"VDC\""
-			(at 44.45 88.9 0)
-			(effects
-				(font
+			(at 64.77 83.82 0)
+			(effects
+				(font

Commit message: Yippiieeeee
Parts:
- added X1: Logo, Vortac:VORTAC_Logo_Gold, symbol Vortac:VORTAC_Logo
Changed lines of the file:
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@@
+	)
+	(symbol
+		(lib_id "Vortac:VORTAC_Logo")
+		(at 113.03 81.28 0)
+		(unit 1)
+		(exclude_from_sim no)
+		(in_bom yes)
+		(on_board yes)
+		(dnp no)
+		(fields_autoplaced yes)
+		(property "Reference" "X1"
+			(at 119.38 79.747 0)
+			(effects
+				(font
+					(size 1.27 1.27)
+				)
+				(justify left)
+			)
+		)
+		(property "Value" "Logo"
+			(at 119.38 82.287 0)
+			(effects
+				(font
+					(size 1.27 1.27)
+				)
+				(justify left)
+			)
+		)
+		(property "Footprint" "Vortac:VORTAC_Logo_Gold"
+			(at 113.03 81.28 0)
+			(effects
+				(font
+					(size 1.27 1.27)
+				)
+				(hide yes)
+			)
+		)
+		(property "Datasheet" ""
+			(at 113.03 81.28 0)
+			(effects
+				(font
+					(size 1.27 1.27)
+				)
+				(hide yes)
+			)
+		)
+		(property "Description" ""
+			(at 113.03 81.28 0)
+			(effects
+				(font
+					(size 1.27 1.27)
+				)
+				(hide yes)
+			)
+		)
+		(instances
+			(project ""
+				(path "/3fc99e24-c24b-45f1-84c7-8e09f231367f"
+					(reference "X1")
+					(unit 1)
+				)
+			)
+		)
 	)
 	(symbol
